File: RelayBoard/RelayBoard.sch (EAGLE design)
At the start: 95 parts, among them IC1 MCP2551/SN RSC 402-904, IC2 MCP2515-I/SOGRB2 RSC 628-3548, U1 CD74HC4067SM96, U2 LM1084IS-3.3, U3 CD74HC4067SM96, U4 ADS1115IDGST, U6 LM1084IS-3.3, U7 LM1084IS-3.3, X1 332-50, X2 332-46

Commit message: remove: - ioexpanders add:       - tm4c129 mcu                - plus two multiplexer and two BNC connector                - 139x115mm board size
Parts:
- removed C10: 100nF, eagle-ltspice:CC0402
- removed IC2: MCP2515-I/SOGRB2 RSC 628-3548, mcp2515:MCP2515-I/SOGRB2
- removed R16, R17, R18, R19: (no value), resistor:R-EU_R0402
- removed R39: 4k7, resistor:R-EU_R0402
- removed R49: 10k, resistor:R-EU_R0402
- removed TP1, TP2, TP3, TP4: TPTP09R, testpad:TPTP09R
- removed U$3, U$4, U$5, U$6, U$7: MCP23016-I/SO, Port Expander:MCP23016-I/SO
- removed XTAL1: 7M-16.000MAAJ-T, TXC-7M-16.000MAAJ-T:7M-16.000MAAJ-T
- added C13, C14, C16, C17, C18, C19, C20: 0.1uF, rcl:C-EUC0402K
- added C15: 2.2uF, rcl:C-EUC0402K
- added C36, C6: 12pF, rcl:C-EUC0402K
- added C37: 0.1uF, eagle-ltspice:CC0402
- added J4: JTAG_ARM_10PIN, MRDT-Connectors:JTAG_ARM_10PIN
- added JP7: (no value), pinhead:PINHD-2X18
- added S2: SWITCH_TACTILE, MRDT-UserInput:SWITCH_TACTILE
- added U5: CD74HC4067SM96, MUX:CD74HC4067SM96
- added U8: TM4C1294NCPDT, MRDT-Microcontrollers:TM4C1294NCPDT
- added X3, X4: A1944-50, con-coax:A1944-50
- added Y3: NX3225GA, MRDT-Passives:NX3225GA
- added Y4: CRYATL_32K_SMD, MRDT-Passives:CRYATL_32K_SMD
- C3, C9: value 22pF -> 12pF; device eagle-ltspice:CC0402 -> rcl:C-EUC0402K
- JP6: device SparkFun-Connectors:M04LOCK_LONGPADS -> pinhead:PINHD-2X30
- R10, R13, R14, R15, R9: value (none) -> 4.7k
- R20: value (none) -> 1M; device resistor:R-EU_R0402 -> rcl:R-EU_R0402
- R21: value (none) -> 51; device resistor:R-EU_R0402 -> rcl:R-EU_R0402
- R22: value (none) -> 4.87k 1%; device resistor:R-EU_R0402 -> rcl:R-EU_R0402
- R23: value (none) -> 2k; device resistor:R-EU_R0402 -> rcl:R-EU_R0402
- R24: value (none) -> 100; device resistor:R-EU_R0402 -> rcl:R-EU_R0402
- R25: value (none) -> 10k; device resistor:R-EU_R0402 -> rcl:R-EU_R0402
- U4: value ADS1115IDGST -> CD74HC4067SM96; device ADC:ADS1115IDGST -> MUX:CD74HC4067SM96
- X1: value 332-50 -> A1944-50; device con-garry:332-50 -> con-coax:A1944-50
- X2: value 332-46 -> A1944-50; device con-garry:332-46 -> con-coax:A1944-50
Connections:
- removed net CAN_INT: IC2.INT
- removed net D28: U$4.GP0.5, X1-14.S
- removed net D29: U$4.GP0.4, X1-13.S
- removed net D30: U$4.GP0.7, X1-12.S
- removed net D31: U$4.GP0.6, X1-11.S
- removed net D32: U$5.GP1.1, X1-10.S
- removed net D33: U$5.GP1.0, X1-9.S
- removed net D34: U$5.GP1.3, X1-8.S
- removed net D35: U$5.GP1.2, X1-7.S
- removed net D36: U$5.GP1.5, X1-6.S
- removed net D37: U$5.GP1.4, X1-5.S
- removed net D38: U$5.GP1.7, X1-4.S
- removed net D39: U$5.GP1.6, X1-3.S
- removed net D40: U$5.GP0.1, X2-42.S
- removed net D41: U$5.GP0.0, X2-41.S
- removed net D42: U$5.GP0.3, X2-40.S
- removed net D43: U$5.GP0.2, X2-39.S
- removed net D44: U$5.GP0.5, X2-38.S
- removed net D45: U$5.GP0.4, X2-37.S
- removed net D46: U$5.GP0.7, X2-36.S
- removed net D47: U$5.GP0.6, X2-35.S
- removed net D48: U$6.GP1.1, X2-34.S
- removed net D49: U$6.GP1.0, X2-33.S
- removed net D50: U$6.GP1.3, X2-32.S
- removed net D51: U$6.GP1.2, X2-31.S
- removed net D52: U$6.GP1.5, X2-30.S
- removed net D53: U$6.GP1.4, X2-29.S
- removed net D54: U$6.GP1.7, X2-28.S
- removed net D55: U$6.GP1.6, X2-27.S
- removed net D56: U$6.GP0.1, X2-26.S
- removed net D57: U$6.GP0.0, X2-25.S
- removed net D58: U$6.GP0.3, X2-24.S
- removed net D59: U$6.GP0.2, X2-23.S
- removed net D60: U$6.GP0.5, X2-22.S
- removed net D61: U$6.GP0.4, X2-21.S
- removed net D62: U$6.GP0.7, X2-20.S
- removed net D63: U$6.GP0.6, X2-19.S
- removed net M2S03: U$7.GP1.7
- removed net N$10: C9.1, IC2.OSC2, XTAL1.1
- removed net N$11: R16.1, U$4.A2
- removed net N$12: R23.1, U$7.A0
- removed net N$13: R24.1, U$7.A1
- removed net N$14: R25.1, U$7.A2
- removed net N$15: R20.1, U$6.A0
- removed net N$16: R21.1, U$6.A1
- removed net N$17: R22.1, U$6.A2
- removed net N$21: R9.1, U$5.A0
- removed net N$22: R10.1, U$5.A1
- removed net N$24: R13.1, U$5.A2
- removed net N$26: R17.1, U$3.A0
- removed net N$27: R18.1, U$3.A1
- removed net N$28: R19.1, U$3.A2
- removed net N$37: U$3.TP
- removed net N$38: TP1.TP, U$6.TP
- removed net N$39: U$7.GP0.5
- removed net N$4: R14.1, U$4.A0
- removed net N$40: U$7.GP0.6
- removed net N$41: U$7.GP0.7
- removed net N$49: IC2.RESET, R39.2
- removed net N$6: R15.1, U$4.A1
- removed net N$7: TP3.TP, U$5.TP
- removed net N$8: TP4.TP, U$4.TP
- removed net N$9: C3.1, IC2.OSC1, XTAL1.3
- new net !RESET: J4.!RESET, R15.1, R24.2, S2.1@A, S2.1@B
- new net +3V3: C16.1, C17.1, C18.1, C19.1, J4.VTARGET, R20.2, R21.2, R25.1, U8G$2.VDD@101, U8G$2.VDD@113, U8G$2.VDD@122, U8G$2.VDD@16, U8G$2.VDD@26, U8G$2.VDD@28, U8G$2.VDD@39, U8G$2.VDD@47, U8G$2.VDD@51, U8G$2.VDD@52, U8G$2.VDD@69, U8G$2.VDD@7, U8G$2.VDD@79, U8G$2.VDD@90, U8G$2.VDDA@8, U8G$2.VREFA+@9
- new net EN0LED0: U8G$1.PF0@42
- new net EN0LED1: U8G$1.PF4@46
- new net EN0RXI_N: U8G$2.EN0RXIN@53
- new net EN0RXI_P: U8G$2.EN0RXIP@54
- new net EN0TXO_N: U8G$2.EN0TXON@56
- new net EN0TXO_P: U8G$2.EN0TXOP@57
- new net N_$2: C20.1, R21.1, U8G$2.VBAT@68
- new net N_$24: R20.1, U8G$2.!WAKE@64
- new net N_$28: C13.1, C14.1, C15.1, U8G$2.VDDC@115, U8G$2.VDDC@87
- new net N_$29: R22.2, U8G$2.RBIAS@59
- new net N_$30: R23.2, U8G$2.OSC1@89
- new net N_$31: C36.1, U8G$2.OSC0@88, Y3.OSC1
- new net N_$32: C9.1, R23.1, Y3.OSC0
- new net N_$33: C37.1, R24.1, R25.2, U8G$2.!RESET@70
- new net N_$34: C6.1, U8G$2.XOSC0@66, Y4.P$1
- new net N_$35: C3.1, U8G$2.XOSC1@67, Y4.P$2
- new net TARGET_TCK/SWCLK: J4.TCK, R10.1, U8G$1.PC0@100
- new net TARGET_TDI: J4.TDI, R14.1, U8G$1.PC2@98
- new net TARGET_TDO/SWO: J4.TDO, R13.1, U8G$1.PC3@97
- new net TARGET_TMS/SWDIO: J4.TMS, R9.1, U8G$1.PC1@99
- net 3.6V: no longer X2-3.S, X2-4.S
- net 5V: no longer X1-49.S, X1-50.S
- net A0: now also U5.I14; no longer U4.AIN1, X1-46.S
- net A1: now also U5.I15; no longer U4.AIN0, X1-45.S
- net A2: now also U5.I12; no longer U4.AIN2, X1-44.S
- net A3: now also U5.I13; no longer U4.AIN3, X1-43.S
- net CAN_CS: no longer IC2.CS
- net CAN_N: no longer X2-17.S
- net CAN_P: no longer X2-18.S
- net CS: no longer X2-14.S
- net D0: now also U5.I10; no longer U$3.GP1.1, X1-42.S
- net D1: now also U5.I11; no longer U$3.GP1.0, X1-41.S
- net D10: now also U5.I0; no longer U$3.GP0.3, X1-32.S
- net D11: now also U5.I1; no longer U$3.GP0.2, X1-31.S
- net D12: now also U4.I14; no longer U$3.GP0.5, X1-30.S
- net D13: now also U4.I15; no longer U$3.GP0.4, X1-29.S
- net D14: now also U4.I12; no longer U$3.GP0.7, X1-28.S
- net D15: now also U4.I13; no longer U$3.GP0.6, X1-27.S
- net D16: now also U4.I10; no longer U$4.GP1.1, X1-26.S
- net D17: now also U4.I11; no longer U$4.GP1.0, X1-25.S
- net D18: now also U4.I8; no longer U$4.GP1.3, X1-24.S
- net D19: now also U4.I9; no longer U$4.GP1.2, X1-23.S
- net D2: now also U5.I8; no longer U$3.GP1.3, X1-40.S
- net D20: now also U4.I1; no longer U$4.GP1.5, X1-22.S
- net D21: now also U4.I0; no longer U$4.GP1.4, X1-21.S
- net D22: now also U4.I3; no longer U$4.GP1.7, X1-20.S
- net D23: now also U4.I2; no longer U$4.GP1.6, X1-19.S
- net D24: now also U4.I5; no longer U$4.GP0.1, X1-18.S
- net D25: now also U4.I4; no longer U$4.GP0.0, X1-17.S
- net D26: now also U4.I7; no longer U$4.GP0.3, X1-16.S
- net D27: now also U4.I6; no longer U$4.GP0.2, X1-15.S
- net D3: now also U5.I9; no longer U$3.GP1.2, X1-39.S
- net D4: now also U5.I5; no longer U$3.GP1.5, X1-38.S
- net D5: now also U5.I4; no longer U$3.GP1.4, X1-37.S
- net D6: now also U5.I7; no longer U$3.GP1.7, X1-36.S
- net D7: now also U5.I6; no longer U$3.GP1.6, X1-35.S
- net D8: now also U5.I2; no longer U$3.GP0.1, X1-34.S
- net D9: now also U5.I3; no longer U$3.GP0.0, X1-33.S
- net DUT_CONNECT: no longer U$7.GP0.3
- net GND: now also C13.2, C14.2, C15.2, C16.2, C17.2, C18.2, C19.2, C20.2, C36.2, C37.2, C6.2, J4.!EXTDBG, J4.GND, R22.1, S2.0@A, S2.0@B, U4.~E, U5.GND, U5.~E, U8G$2.GND@114, U8G$2.GND@17, U8G$2.GND@48, U8G$2.GND@55, U8G$2.GND@58, U8G$2.GND@80, U8G$2.GNDA@10, X1.2, X2.2, X3.2, X4.2; no longer C10.2, IC2.VSS, JP6.2, JP6.4, R13.2, R15.2, R16.2, R17.2, R18.2, R19.2, R20.2, R21.2, R23.2, R9.2, U$3.VSS, U$3.VSS_2, U$3.VSS_3, U$4.VSS, U$4.VSS_2, U$4.VSS_3, U$5.VSS, U$5.VSS_2, U$5.VSS_3, U$6.VSS, U$6.VSS_2, U$6.VSS_3, U$7.VSS, U$7.VSS_2, U$7.VSS_3, U4.ADDR, X1-1.S, X1-2.S, X2-1.S, X2-2.S, X2-45.S, X2-46.S
- net IO_INT: no longer R49.1, U$3.~INT, U$4.~INT, U$5.~INT, U$6.~INT, U$7.~INT
- net M1OUT: now also U4.COMMON_IN/OUT, X1.1; no longer JP6.1
- net M1S0: now also U4.S0; no longer U$7.GP1.0
- net M1S1: now also U4.S1; no longer U$7.GP1.1
- net M1S2: now also U4.S2; no longer U$7.GP1.2
- net M1S3: now also U4.S3; no longer U$7.GP1.3
- net M2OUT: now also U5.COMMON_IN/OUT, X2.1; no longer JP6.3
- net M2S0: now also U5.S0; no longer U$7.GP1.4
- net M2S1: now also U5.S1; no longer U$7.GP1.5
- net M2S2: now also U5.S2; no longer U$7.GP1.6
- net M2S3: now also U5.S3
- net MISO: no longer IC2.SO, X2-12.S
- net MOSI: no longer IC2.SI, X2-13.S
- net N$2: now also R10.2, R13.2, R14.2, R15.2, R9.2; no longer TP2.TP, U$7.TP
- net N$45: no longer IC2.RXCAN
- net N$47: no longer IC2.TXCAN
- net NRESET: no longer X2-8.S
- net ONEWIRE: no longer X2-7.S
- net PROGRAM: no longer U$7.GP0.4
- net RX: now also J4.P$7, U8G$1.PA0@33; no longer X2-6.S
- net SCK: no longer IC2.SCK
- net SCL: no longer X2-15.S
- net SCLK: no longer X2-11.S
- net SDA: no longer X2-16.S
- net SWDCLK: no longer X2-10.S
- net SWDIO: no longer X2-9.S
- net TEST_FAIL: no longer U$7.GP0.2
- net TEST_PASS: no longer U$7.GP0.1
- net TEST_RUN: no longer U$7.GP0.0
- net TFT_SCL: no longer U$3.SCL, U$4.SCL, U$5.SCL, U$6.SCL, U$7.SCL, U4.SCL
- net TFT_SDA: no longer U$3.SDA, U$4.SDA, U$5.SDA, U$6.SDA, U$7.SDA, U4.SDA
- net TX: now also J4.GND1, U8G$1.PA1@34; no longer X2-5.S
- net VCC: now also U5.VCC; no longer C10.1, IC2.VDD, R10.2, R14.2, R22.2, R24.2, R25.2, R39.1, R49.2, U$3.VDD, U$4.VDD, U$5.VDD, U$6.VDD, U$7.VDD, U4.VDD, X1-47.S, X1-48.S
Other:
- note added: "Ethernet Activity LED"
- note added: "Ethernet Link LED"
- note added: "GPIO"
- note added: "JTAG Signals"
- note added: "Serial0 back to programmer"

Commit message: additions
- common connector for isp, jtag, swd
- change LDOs to the one which have Enable pin
- UART -> USB interface and isolator to the uart side
- dedicated MCU supply
Parts:
- removed C7, C8: 10uF, rcl:C-EUC0402
- removed JP30: RASPBERRYPI-B+-GPIO, SparkFun-Boards:RASPBERRYPI-B+-GPIO
- removed R11, R12, R31, R32, R4: (no value), resistor:R-EU_R0402
- removed U7: LM1084IS-3.3, LDO:LM1084IS-3.3
- added C10, C12, C21, C22, C39, C45: 0.1uF, rcl:C-EUC0402
- added C23, C24: 1uF, rcl:C-EUC0402
- added C25, C26, C49: 10uF, rcl:C-EUC0402
- added ISP1: AVRISP-6, JDT-1800_smahed:AVRISP-6
- added J1: JTAG_ARM_10PIN, MRDT-Connectors:JTAG_ARM_10PIN
- added JP8: USB-B, SparkFun-Connectors:USBPTH
- added LED9: (no value), JDT-1800_smahed:LEDCHIP-LED0805
- added R100, R101, R102, R103, R104, R105, R106, R107, R108, R109, R110, R111, R112, R113, R114, R115, R117, R118, R119, R120, R121, R122, R123, R124, R125, R126, R127, R128, R129, R130, R131, R132, R133, R134, R135, R18, R19, R39, R49, R51, R52, R53, R54, R55, R56, R57, R58, R59, R60, R61, R62, R63, R64, R65, R66, R67, R68, R69, R70, R71, R72, R73, R74, R75, R76, R77, R78, R79, R80, R81, R82, R83, R84, R85, R86, R87, R88, R89, R90, R91, R92, R93, R94, R95, R96, R97, R98, R99: 200R, resistor:R-EU_R0402
- added R116, R136, R137, R138, R139: (no value), resistor:R-EU_R0402
- added R16, R17: (no value), JDT-1800_smahed:R-US_R5025
- added U$1, U$10, U$11, U$12, U$13, U$14, U$15, U$16, U$17, U$18, U$19, U$2, U$20, U$21, U$22, U$23, U$24, U$25, U$26, U$27, U$28, U$29, U$3, U$30, U$31, U$32, U$33, U$35, U$36, U$37, U$38, U$39, U$4, U$40, U$41, U$42, U$43, U$44, U$45, U$46, U$47, U$48, U$49, U$50, U$6, U$7, U$8, U$9: zener_3.3V, SparkFun-DiscreteSemi:MMBZ27VCLT1
- added U$34: MCP1703T-3302E/CB, MCP1703:MCP1703T-3302E/CB
- added U10, U11, U12, U9: INA219AIDCNR, INA219:INA219AIDCNR
- added U13: FT230XQ, ftdichip:FT230XQ
- added U14: ADUM1201ARZ, ADUM1201ARZ:ADUM1201ARZ
- added U16: TL1963AKTTR., TL1963:TL1963AKTTR.
- C2, C4, C5: value 0.1uF -> 10uF
- R1, R38: value (none) -> 22R; device resistor:R-EU_R0402 -> SparkFun-Passives:RESISTOR0402-RES
- R34, R42, R43, R45, R50: value 0R -> 200R
- R47, R48: value 10k -> 200R
- R5, R6: value 0R -> (none); device resistor:R-EU_R0402 -> JDT-1800_smahed:R-US_R5025
- U2, U6: value LM1084IS-3.3 -> TL1963AKTTR.; device LDO:LM1084IS-3.3 -> TL1963:TL1963AKTTR.
Connections:
- removed net +3V3: C16.1, C17.1, C18.1, C19.1, J4.VTARGET, R20.2, R21.2, R25.1, U8G$2.VDD@101, U8G$2.VDD@113, U8G$2.VDD@122, U8G$2.VDD@16, U8G$2.VDD@26, U8G$2.VDD@28, U8G$2.VDD@39, U8G$2.VDD@47, U8G$2.VDD@51, U8G$2.VDD@52, U8G$2.VDD@69, U8G$2.VDD@7, U8G$2.VDD@79, U8G$2.VDD@90, U8G$2.VDDA@8, U8G$2.VREFA+@9
- removed net 3.6V: C8.1, R31.2, R33.2, U7.OUT, U7.VOUT
- removed net 5V: C1.1, JP30.5V@2, JP30.5V@4, R11.2, R29.2, U2.OUT, U2.VOUT
- removed net A0: U3.I14, U5.I14
- removed net A1: U3.I15, U5.I15
- removed net A2: U3.I12, U5.I12
- removed net A3: U3.I13, U5.I13
- removed net ADJ: R3.2, R4.1, U6.ADJ/GND
- removed net ADJ1: R11.1, R12.2, U2.ADJ/GND
- removed net ADJ2: R31.1, R32.2, U7.ADJ/GND
- removed net CAN_CS: JP30.CE1, R48.2
- removed net D0: U3.I10, U5.I10
- removed net D1: U3.I11, U5.I11
- removed net D10: U3.I0, U5.I0
- removed net D11: U3.I1, U5.I1
- removed net D12: U1.I14, U4.I14
- removed net D13: U1.I15, U4.I15
- removed net D14: U1.I12, U4.I12
- removed net D15: U1.I13, U4.I13
- removed net D16: U1.I10, U4.I10
- removed net D17: U1.I11, U4.I11
- removed net D18: U1.I8, U4.I8
- removed net D19: U1.I9, U4.I9
- removed net D2: U3.I8, U5.I8
- removed net D20: U1.I1, U4.I1
- removed net D21: U1.I0, U4.I0
- removed net D22: U1.I3, U4.I3
- removed net D23: U1.I2, U4.I2
- removed net D24: U1.I5, U4.I5
- removed net D25: U1.I4, U4.I4
- removed net D26: U1.I7, U4.I7
- removed net D27: U1.I6, U4.I6
- removed net D3: U3.I9, U5.I9
- removed net D4: U3.I5, U5.I5
- removed net D5: U3.I4, U5.I4
- removed net D6: U3.I7, U5.I7
- removed net D7: U3.I6, U5.I6
- removed net D8: U3.I2, U5.I2
- removed net D9: U3.I3, U5.I3
- removed net IO_INT: JP30.GP17
- removed net NC0: JP30.3.3V@1
- removed net RPI_NRESET: JP30.GP18#, R34.2
- removed net RPI_SWDCLK: JP30.GP25, R5.2
- removed net RPI_SWDIO: JP30.GP24, R6.2
- removed net RX: J4.P$7, JP3.10, R38.1, U8G$1.PA0@33
- removed net SCK: R45.1
- removed net TARGET_CS: JP30.GP4, R47.2, R50.2
- removed net TFT_CS: JP30.CE0
- removed net TFT_MISO: JP30.MISO, R43.2
- removed net TFT_MOSI: JP30.MOSI, R42.2
- removed net TFT_RX: JP30.TXO, R37.2
- removed net TFT_SCK: JP30.SCLK, R45.2
- removed net TFT_SCL: JP30.SCL, R1.1, R35.2
- removed net TFT_SDA: JP30.SDA, R2.1, R36.2
- removed net TFT_TX: JP30.RXI, R38.2
- removed net TX: J4.GND1, JP3.11, R37.1, U8G$1.PA1@34
- removed net VOLTAGE_INPUT: C2.1, C4.1, C5.1, JP5.PWR, U2.IN, U6.IN, U7.IN
- new net ADJ3: R2.1, R35.2, U16.SENSE/ADJ
- new net ADJ4: R116.2, R37.1, U2.SENSE/ADJ
- new net ADJ5: R137.1, R138.2, U6.SENSE/ADJ
- new net DUT_SH+: R17.2, U12.VIN+
- new net DUT_SH_-: R17.1, U12.VIN-
- new net HOST_GND: C39.1, C45.1, C49.1, U13.GND, U13.GND@1, U14.GND2
- new net HOST_UART_RX: U13.RXD, U14.VOB
- new net HOST_UART_TX: U13.TXD, U14.VOA
- new net LDO1: R108.1, R16.2, R29.2, R60.2, U$22.A1, U$22.A2, U11.VIN-
- new net LDO1_ENABLE: R36.1, U16.!SHDN
- new net LDO1_SH+: C1.1, R16.1, R2.2, U11.VIN+, U16.OUT
- new net LDO2: R109.1, R30.2, R6.2, R61.2, U$23.A1, U$23.A2, U10.VIN-
- new net LDO2_ENABLE: R136.1, U2.!SHDN
- new net LDO2_SH+: C2.1, R37.2, R6.1, U10.VIN+, U2.OUT
- new net LDO3: R110.1, R33.2, R5.2, R62.2, U$24.A1, U$24.A2, U9.VIN-
- new net LDO3_ENABLE: R139.1, U6.!SHDN
- new net LDO3_SH+: C4.1, R137.2, R5.1, U6.OUT, U9.VIN+
- new net M0S0: U4.S0
- new net M0S1: U4.S1
- new net M0S2: U4.S2
- new net M0S3: U4.S3
- new net M3S0: U5.S0
- new net M3S1: U5.S1
- new net M3S2: U5.S2
- new net M3S3: U5.S3
- new net N$10: JP6.11, R43.1
- new net N$100: JP6.38, R106.2
- new net N$101: JP6.40, R107.2
- new net N$102: JP6.42, R108.2
- new net N$103: JP6.44, R109.2
- new net N$104: JP6.46, R110.2
- new net N$105: JP6.48, R111.2
- new net N$106: JP6.50, R112.2
- new net N$107: JP6.52, R113.2
- new net N$108: JP6.54, R114.2
- new net N$109: JP6.56, R115.2
- new net N$11: JP6.13, R45.1
- new net N$110: LED9.A, R3.1
- new net N$111: JP6.60, R117.2
- new net N$112: R18.2, U$12.A2
- new net N$113: R87.2, U$25.A2
- new net N$114: R88.1, U$12.A1
- new net N$115: R89.1, U$11.A1
- new net N$116: R19.2, U$11.A2
- new net N$117: R90.1, U$10.A1
- new net N$118: R34.2, U$10.A2
- new net N$119: R91.1, U$9.A1
- new net N$12: JP6.15, R47.1
- new net N$120: R39.2, U$9.A2
- new net N$121: R92.1, U$8.A1
- new net N$122: R42.2, U$8.A2
- new net N$123: R43.2, U$7.A2
- new net N$124: R93.1, U$7.A1
- new net N$125: R94.1, U$6.A1
- new net N$126: R45.2, U$6.A2
- new net N$127: R47.2, U$4.A2
- new net N$128: R95.1, U$4.A1
- new net N$129: R96.1, U$3.A1
- new net N$13: JP6.17, R48.1
- new net N$130: R48.2, U$3.A2
- new net N$131: R97.1, U$2.A1
- new net N$132: R49.2, U$2.A2
- new net N$133: R50.2, U$1.A2
- new net N$134: R98.1, U$1.A1
- new net N$135: R99.1, U$13.A1
- new net N$136: R51.2, U$13.A2
- new net N$137: R52.2, U$14.A2
- new net N$138: R100.1, U$14.A1
- new net N$139: R101.1, U$15.A1
- new net N$14: JP6.19, R49.1
- new net N$140: R53.2, U$15.A2
- new net N$141: R54.2, U$16.A2
- new net N$142: R102.1, U$16.A1
- new net N$143: R55.2, U$17.A2
- new net N$144: R103.1, U$17.A1
- new net N$145: R104.1, U$18.A1
- new net N$146: R56.2, U$18.A2
- new net N$147: R105.1, U$19.A1
- new net N$148: R57.2, U$19.A2
- new net N$149: R106.1, U$20.A1
- new net N$15: JP6.21, R50.1
- new net N$150: R58.2, U$20.A2
- new net N$151: R59.2, U$21.A2
- new net N$152: R107.1, U$21.A1
- new net N$157: R135.1, U$25.A1
- new net N$159: C39.2, U13.3V3OUT
- new net N$16: JP6.23, R51.1
- new net N$160: R134.1, U$26.A1
- new net N$161: R86.2, U$26.A2
- new net N$162: R85.2, U$48.A2
- new net N$163: R133.1, U$48.A1
- new net N$164: R84.2, U$47.A2
- new net N$165: R83.2, U$46.A2
- new net N$166: R82.2, U$45.A2
- new net N$167: R81.2, U$44.A2
- new net N$168: R80.2, U$43.A2
- new net N$169: R79.2, U$42.A2
- new net N$17: JP6.25, R52.1
- new net N$170: R78.2, U$41.A2
- new net N$171: R77.2, U$40.A2
- new net N$172: R76.2, U$39.A2
- new net N$173: R75.2, U$38.A2
- new net N$174: R73.2, U$28.A2
- new net N$175: R72.2, U$29.A2
- new net N$176: R71.2, U$30.A2
- new net N$177: R70.2, U$31.A2
- new net N$178: R69.2, U$32.A2
- new net N$179: R68.2, U$33.A1
- new net N$18: JP6.27, R53.1
- new net N$180: R67.2, U$35.A2
- new net N$181: R66.2, U$36.A2
- new net N$182: R129.1, U$44.A1
- new net N$183: R132.1, U$47.A1
- new net N$184: R131.1, U$46.A1
- new net N$185: R130.1, U$45.A1
- new net N$186: R74.2, U$27.A2
- new net N$187: R128.1, U$43.A1
- new net N$188: R127.1, U$42.A1
- new net N$189: R65.2, U$37.A2
- new net N$19: JP6.29, R54.1
- new net N$190: R64.2, U$49.A2
- new net N$191: R63.2, U$50.A2
- new net N$192: R126.1, U$41.A1
- new net N$193: R125.1, U$40.A1
- new net N$194: R124.1, U$39.A1
- new net N$195: R123.1, U$38.A1
- new net N$196: R122.1, U$27.A1
- new net N$197: R121.1, U$28.A1
- new net N$198: R120.1, U$29.A1
- new net N$199: R119.1, U$30.A1
- new net N$20: JP6.31, R55.1
- new net N$200: R118.1, U$31.A1
- new net N$201: R117.1, U$32.A1
- new net N$203: R115.1, U$33.A2
- new net N$204: R114.1, U$36.A1
- new net N$205: R113.1, U$37.A1
- new net N$206: R112.1, U$49.A1
- new net N$207: R111.1, U$50.A1
- new net N$21: JP6.33, R56.1
- new net N$216: C23.1, U$34.VIN
- new net N$22: JP6.35, R57.1
- new net N$24: JP6.37, R58.1
- new net N$26: JP6.39, R59.1
- new net N$27: JP6.41, R60.1
- new net N$28: JP6.43, R61.1
- new net N$29: JP6.45, R62.1
- new net N$30: JP6.47, R63.1
- new net N$31: JP6.49, R64.1
- new net N$32: JP6.51, R65.1
- new net N$37: JP6.53, R66.1
- new net N$38: JP6.55, R67.1
- new net N$39: JP6.57, R68.1
- new net N$4: JP6.1, R18.1
- new net N$40: JP6.59, R69.1
- new net N$41: JP7.1, R70.1
- new net N$42: JP7.3, R71.1
- new net N$43: JP7.5, R72.1
- new net N$49: JP7.7, R73.1
- new net N$50: JP7.9, R74.1
- new net N$51: JP7.11, R75.1
- new net N$52: JP7.13, R76.1
- new net N$53: JP7.15, R77.1
- new net N$54: JP7.17, R78.1
- new net N$55: JP7.19, R79.1
- new net N$56: JP7.21, R80.1
- new net N$57: JP7.23, R81.1
- new net N$58: JP7.25, R82.1
- new net N$59: JP7.27, R83.1
- new net N$6: JP6.3, R19.1
- new net N$60: JP7.29, R84.1
- new net N$61: JP7.31, R85.1
- new net N$62: JP7.33, R86.1
- new net N$63: JP7.35, R87.1
- new net N$64: JP7.2, R118.2
- new net N$65: JP7.4, R119.2
- new net N$66: JP7.6, R120.2
- new net N$67: JP7.8, R121.2
- new net N$68: JP7.10, R122.2
- new net N$69: JP7.12, R123.2
- new net N$7: JP6.5, R34.1
- new net N$70: JP7.14, R124.2
- new net N$71: JP7.16, R125.2
- new net N$72: JP7.18, R126.2
- new net N$73: JP7.20, R127.2
- new net N$74: JP7.22, R128.2
- new net N$75: JP7.24, R129.2
- new net N$76: JP7.26, R130.2
- new net N$77: JP7.28, R131.2
- new net N$78: JP7.30, R132.2
- new net N$79: JP7.32, R133.2
- new net N$8: JP6.7, R39.1
- new net N$80: JP7.34, R134.2
- new net N$81: JP7.36, R135.2
- new net N$82: JP6.2, R88.2
- new net N$83: JP6.4, R89.2
- new net N$84: JP6.6, R90.2
- new net N$85: JP6.8, R91.2
- new net N$86: JP6.10, R92.2
- new net N$87: JP6.12, R93.2
- new net N$88: JP6.14, R94.2
- new net N$89: JP6.16, R95.2
- new net N$9: JP6.9, R42.1
- new net N$90: JP6.18, R96.2
- new net N$91: JP6.20, R97.2
- new net N$92: JP6.22, R98.2
- new net N$93: JP6.24, R99.2
- new net N$94: JP6.26, R100.2
- new net N$95: JP6.28, R101.2
- new net N$96: JP6.30, R102.2
- new net N$97: JP6.32, R103.2
- new net N$98: JP6.34, R104.2
- new net N$99: JP6.36, R105.2
- new net POWER_IN: C25.1, C26.1, C5.1, JP5.PWR, U16.IN, U2.IN, U6.IN
- new net SWDCLK/TCLK/SCK: ISP1.SCK, J1.TCK, JP2.9
- new net SWDIO/TMS: J1.TMS, JP2.7
- new net SWO/TDO/MISO: ISP1.MISO, J1.TDO, JP2.13
- new net TDI/MISO: JP2.5
- new net TDI/MOSI: ISP1.MOSI, J1.TDI
- new net TRST_3V3: R136.2, R139.2, R36.2
- new net TSTR_3V3: C10.1, C12.1, C16.1, C17.1, C18.1, C19.1, C21.1, C22.2, C24.1, ISP1.VCC, J1.VTARGET, J4.VTARGET, R20.2, R21.2, R25.1, R3.2, U$34.VOUT, U10.A1, U10.VS, U11.A0, U11.VS, U12.VS, U14.VDD1, U8G$2.VDD@101, U8G$2.VDD@113, U8G$2.VDD@122, U8G$2.VDD@16, U8G$2.VDD@26, U8G$2.VDD@28, U8G$2.VDD@39, U8G$2.VDD@47, U8G$2.VDD@51, U8G$2.VDD@52, U8G$2.VDD@69, U8G$2.VDD@7, U8G$2.VDD@79, U8G$2.VDD@90, U8G$2.VDDA@8, U8G$2.VREFA+@9, U9.A0, U9.A1, U9.VS
- new net TSTR_RX: J4.P$7, JP3.10, U14.VIA, U8G$1.PA0@33
- new net TSTR_SCL: U10.SCL, U11.SCL, U12.SCL, U9.SCL
- new net TSTR_SDA: U10.SDA, U11.SDA, U12.SDA, U9.SDA
- new net TSTR_TX: J4.GND1, JP3.11, U14.VIB, U8G$1.PA1@34
- new net USBD_N: R38.2, U13.USBDM
- new net USBD_P: R1.2, U13.USBDP
- new net USB_N: JP8.D-, R38.1
- new net USB_P: JP8.D+, R1.1
- new net VBUS: C45.2, C49.2, JP8.VBUS, U13.VCC, U13.VCCIO, U14.VDD2
- net CS: no longer R50.1
- net GND: now also C10.2, C12.2, C21.2, C22.1, C23.2, C24.2, C25.2, C26.2, ISP1.GND, J1.GND, LED9.C, R116.1, R138.1, R35.1, U$1.C, U$10.C, U$11.C, U$12.C, U$13.C, U$14.C, U$15.C, U$16.C, U$17.C, U$18.C, U$19.C, U$2.C, U$20.C, U$21.C, U$22.C, U$23.C, U$24.C, U$25.C, U$26.C, U$27.C, U$28.C, U$29.C, U$3.C, U$30.C, U$31.C, U$32.C, U$33.C, U$34.GND, U$35.C, U$36.C, U$37.C, U$38.C, U$39.C, U$4.C, U$40.C, U$41.C, U$42.C, U$43.C, U$44.C, U$45.C, U$46.C, U$47.C, U$48.C, U$49.C, U$50.C, U$6.C, U$7.C, U$8.C, U$9.C, U10.A0, U10.GND, U11.A1, U11.GND, U12.A0, U12.A1, U12.GND, U14.GND1, U16.GND, U16.GND_2, U2.GND, U2.GND_2, U6.GND, U6.GND_2, U9.GND; no longer C7.2, C8.2, JP30.GND@14, JP30.GND@20, JP30.GND@25, JP30.GND@30, JP30.GND@34, JP30.GND@39, JP30.GND@6, JP30.GND@9, R12.1, R3.1, R32.1
- net M1S0: no longer U4.S0
- net M1S1: no longer U4.S1
- net M1S2: no longer U4.S2
- net M1S3: no longer U4.S3
- net M2S0: no longer U5.S0
- net M2S1: no longer U5.S1
- net M2S2: no longer U5.S2
- net M2S3: no longer U5.S3
- net MISO: no longer R43.1
- net MOSI: no longer R42.1
- net NRESET: now also ISP1.RST, J1.!RESET; no longer R34.1
- net SCL: no longer R35.1
- net SDA: no longer R36.1
- net SWDCLK: no longer JP2.9, R5.1
- net SWDIO: no longer JP2.7, R6.1
- net SWO: no longer JP2.13
- net VCC: no longer C7.1, R1.2, R2.2, R30.2, R4.2, R47.1, R48.1, U6.OUT, U6.VOUT
Other:
- note added: "max: 16v 250mA"

Commit message: layout done
Add: - binding posts with 19.05 mm spacing
         - top/bottom  VCC/GND plane
Parts:
- removed C11: 100nF, eagle-ltspice:CC0402
- removed C39, C45: 0.1uF, rcl:C-EUC0402
- removed C49: 10uF, rcl:C-EUC0402
- removed IC1: MCP2551/SN RSC 402-904, microchip-dspic:MCP2551/SN
- removed R120, R121, R122, R123, R124, R125, R126, R127, R128, R88, R89, R90: 200R, resistor:R-EU_R0402
- removed S2: SWITCH_TACTILE, MRDT-UserInput:SWITCH_TACTILE
- removed U$11, U$12, U$27, U$28, U$29, U$30, U$31, U$32, U$33, U$35, U$38, U$39, U$40, U$41, U$42, U$43: zener_3.3V, SparkFun-DiscreteSemi:MMBZ27VCLT1
- removed U13: FT230XQ, ftdichip:FT230XQ
- removed X3: A1944-50, con-coax:A1944-50
- removed Y4: CRYATL_32K_SMD, MRDT-Passives:CRYATL_32K_SMD
- added C7: 10uF, rcl:C-EUC0402K
- added D1: (no value), diode:DIODE-SOD523
- added F1: (no value), fuse:GSH15
- added JP10: DUT_CS_MASTER, SparkFun-Retired:JUMPER-2SMD-NO
- added JP11: (no value), SparkFun:JUMPER-2SMD-NO
- added JP12, JP13: BINDING_POST, SparkFun-Connectors:BINDING_POST
- added JP9: (no value), SparkFun-Retired:JUMPER-2SMD-NC
- added LED10: (no value), JDT-1800_smahed:LEDCHIP-LED0805
- added R11, R12, R31, R32, R4: 4k7, resistor:R-EU_R0402
- added R140: 120, resistor:R-EU_R0402
- added S1: (no value), switch:320-916
- added S3: SWS003, smd-special:SWS003
- added STANDOFF1, STANDOFF2, STANDOFF5, STANDOFF6: STAND-OFF, SparkFun-Electromechanical:STAND-OFF
- added SV1: (no value), con-lstb:MA10-2
- added U$5: zener_3.3V, SparkFun-DiscreteSemi:MMBZ27VCLT1
- added U15: SN65HVD230D, sn65hvd23x:SN65HVD230D
- added U17: FT230XS, FT230XS:FT230XS
- added U7: MCP2003-E/SN, MCP2003-E_SN:MCP2003-E/SN
- C3, C6: value 12pF -> 0.1uF
- JP1: value (none) -> RESET; device JDT-1800_smahed:PINHD-1X6B -> SparkFun-Retired:JUMPER-2SMD-NO
- JP4: value (none) -> DUT_CS_MASTER; device SparkFun:JUMPER-2SMD-NO -> SparkFun-Retired:JUMPER-2SMD-NO
- JP7: value (none) -> DUT_CS_RecieveAllMSG; device pinhead:PINHD-2X18 -> SparkFun-Retired:JUMPER-2SMD-NO
- R117: value 200R -> 1k
- R118, R119, R72, R73, R74, R75, R76, R77: value 200R -> 4k7
- R136, R139, R36: value (none) -> 4k7
- R18, R19, R34, R69, R70, R71, R78, R79, R80, R81: value 200R -> 4.7k
- R40: value 10k -> (none)
- R41: value 120 -> 0R
- R44: value 4k7 -> 0R
- R46: value 18k -> 4.7k
- U5: value CD74HC4067SM96 -> MCP4725A0T-E/CH; device MUX:CD74HC4067SM96 -> MCP4725:MCP4725A0T-E/CH
Connections:
- removed net 5VSUPPLY: JP2.19
- removed net CAN_N: IC1.CANL, JP3.2, R41.2
- removed net CAN_P: IC1.CANH, JP3.1, JP4.1
- removed net CS: JP3.6
- removed net DUT_SH_-: R17.1, U12.VIN-
- removed net EN0LED0: U8G$1.PF0@42
- removed net EN0LED1: U8G$1.PF4@46
- removed net EN0RXI_N: U8G$2.EN0RXIN@53
- removed net EN0RXI_P: U8G$2.EN0RXIP@54
- removed net EN0TXO_N: U8G$2.EN0TXON@56
- removed net EN0TXO_P: U8G$2.EN0TXOP@57
- removed net LIN: JP3.13
- removed net M3S0: U5.S0
- removed net M3S1: U5.S1
- removed net M3S2: U5.S2
- removed net M3S3: U5.S3
- removed net MISO: JP3.4
- removed net MOSI: JP3.7
- removed net N$111: JP6.60, R117.2
- removed net N$113: R87.2, U$25.A2
- removed net N$114: R88.1, U$12.A1
- removed net N$115: R89.1, U$11.A1
- removed net N$116: R19.2, U$11.A2
- removed net N$117: R90.1, U$10.A1
- removed net N$118: R34.2, U$10.A2
- removed net N$119: R91.1, U$9.A1
- removed net N$120: R39.2, U$9.A2
- removed net N$121: R92.1, U$8.A1
- removed net N$122: R42.2, U$8.A2
- removed net N$123: R43.2, U$7.A2
- removed net N$124: R93.1, U$7.A1
- removed net N$125: R94.1, U$6.A1
- removed net N$126: R45.2, U$6.A2
- removed net N$127: R47.2, U$4.A2
- removed net N$128: R95.1, U$4.A1
- removed net N$129: R96.1, U$3.A1
- removed net N$130: R48.2, U$3.A2
- removed net N$131: R97.1, U$2.A1
- removed net N$132: R49.2, U$2.A2
- removed net N$133: R50.2, U$1.A2
- removed net N$134: R98.1, U$1.A1
- removed net N$135: R99.1, U$13.A1
- removed net N$136: R51.2, U$13.A2
- removed net N$137: R52.2, U$14.A2
- removed net N$138: R100.1, U$14.A1
- removed net N$139: R101.1, U$15.A1
- removed net N$140: R53.2, U$15.A2
- removed net N$141: R54.2, U$16.A2
- removed net N$142: R102.1, U$16.A1
- removed net N$143: R55.2, U$17.A2
- removed net N$144: R103.1, U$17.A1
- removed net N$145: R104.1, U$18.A1
- removed net N$146: R56.2, U$18.A2
- removed net N$147: R105.1, U$19.A1
- removed net N$148: R57.2, U$19.A2
- removed net N$149: R106.1, U$20.A1
- removed net N$150: R58.2, U$20.A2
- removed net N$151: R59.2, U$21.A2
- removed net N$152: R107.1, U$21.A1
- removed net N$157: R135.1, U$25.A1
- removed net N$159: C39.2, U13.3V3OUT
- removed net N$160: R134.1, U$26.A1
- removed net N$161: R86.2, U$26.A2
- removed net N$162: R85.2, U$48.A2
- removed net N$163: R133.1, U$48.A1
- removed net N$164: R84.2, U$47.A2
- removed net N$165: R83.2, U$46.A2
- removed net N$166: R82.2, U$45.A2
- removed net N$167: R81.2, U$44.A2
- removed net N$168: R80.2, U$43.A2
- removed net N$169: R79.2, U$42.A2
- removed net N$170: R78.2, U$41.A2
- removed net N$171: R77.2, U$40.A2
- removed net N$172: R76.2, U$39.A2
- removed net N$173: R75.2, U$38.A2
- removed net N$174: R73.2, U$28.A2
- removed net N$175: R72.2, U$29.A2
- removed net N$176: R71.2, U$30.A2
- removed net N$177: R70.2, U$31.A2
- removed net N$178: R69.2, U$32.A2
- removed net N$179: R68.2, U$33.A1
- removed net N$181: R66.2, U$36.A2
- removed net N$182: R129.1, U$44.A1
- removed net N$183: R132.1, U$47.A1
- removed net N$184: R131.1, U$46.A1
- removed net N$185: R130.1, U$45.A1
- removed net N$186: R74.2, U$27.A2
- removed net N$187: R128.1, U$43.A1
- removed net N$188: R127.1, U$42.A1
- removed net N$189: R65.2, U$37.A2
- removed net N$190: R64.2, U$49.A2
- removed net N$191: R63.2, U$50.A2
- removed net N$192: R126.1, U$41.A1
- removed net N$193: R125.1, U$40.A1
- removed net N$194: R124.1, U$39.A1
- removed net N$195: R123.1, U$38.A1
- removed net N$196: R122.1, U$27.A1
- removed net N$197: R121.1, U$28.A1
- removed net N$198: R120.1, U$29.A1
- removed net N$199: R119.1, U$30.A1
- removed net N$200: R118.1, U$31.A1
- removed net N$201: R117.1, U$32.A1
- removed net N$203: R115.1, U$33.A2
- removed net N$204: R114.1, U$36.A1
- removed net N$205: R113.1, U$37.A1
- removed net N$206: R112.1, U$49.A1
- removed net N$207: R111.1, U$50.A1
- removed net N$53: JP7.15, R77.1
- removed net N$54: JP7.17, R78.1
- removed net N$55: JP7.19, R79.1
- removed net N$56: JP7.21, R80.1
- removed net N$57: JP7.23, R81.1
- removed net N$63: JP7.35, R87.1
- removed net N$66: JP7.6, R120.2
- removed net N$67: JP7.8, R121.2
- removed net N$68: JP7.10, R122.2
- removed net N$69: JP7.12, R123.2
- removed net N$70: JP7.14, R124.2
- removed net N$71: JP7.16, R125.2
- removed net N$72: JP7.18, R126.2
- removed net N$73: JP7.20, R127.2
- removed net N$74: JP7.22, R128.2
- removed net N$81: JP7.36, R135.2
- removed net N$82: JP6.2, R88.2
- removed net N$83: JP6.4, R89.2
- removed net N$84: JP6.6, R90.2
- removed net N_$34: C6.1, U8G$2.XOSC0@66, Y4.P$1
- removed net N_$35: C3.1, U8G$2.XOSC1@67, Y4.P$2
- removed net ONEWIRE: JP3.3
- removed net PI_5V: C11.1, IC1.VDD
- removed net POWER_IN: C25.1, C26.1, C5.1, JP5.PWR, U16.IN, U2.IN, U6.IN
- removed net PROGRAM: R28.2
- removed net SCL: JP3.9
- removed net SCLK: JP3.5
- removed net SDA: JP3.8
- removed net SWDCLK: JP1.4
- removed net SWDIO: JP1.5
- removed net SWO: JP1.3
- removed net SWO/TDO/MISO: ISP1.MISO, J1.TDO, JP2.13
- removed net TDI/MOSI: ISP1.MOSI, J1.TDI
- removed net TRST_3V3: R136.2, R139.2, R36.2
- new net AD0: R42.2, U$8.A2, U1.I4, U8G$1.PK3@21
- new net AD1: R92.1, U$8.A1, U1.I3, U8G$1.PK2@20
- new net AD10: R49.2, U$2.A2, U1.I10, U8G$1.PD1@2
- new net AD11: R97.1, U$2.A1, U1.I11, U8G$1.PD0@1
- new net AD12: R50.2, U$1.A2, U1.I12, U8G$1.PD7@128
- new net AD13: R98.1, U$1.A1, U1.I13, U8G$1.PD6@127
- new net AD14: R51.2, U$13.A2, U1.I14, U8G$1.PD5@126
- new net AD15: R99.1, U$13.A1, U1.I15, U8G$1.PD4@125
- new net AD16: R52.2, U$14.A2, U4.I0, U8G$1.PE5@124
- new net AD17: R100.1, U$14.A1, U4.I1, U8G$1.PE4@123
- new net AD18: R53.2, U$15.A2, U4.I2, U8G$1.PB4@121
- new net AD19: R101.1, U$15.A1, U4.I3, U8G$1.PB5@120
- new net AD2: R43.2, U$7.A2, U1.I2, U8G$1.PK1@19
- new net AD3: R93.1, U$7.A1, U1.I1, U8G$1.PK0@18
- new net AD4: R45.2, U$6.A2, U1.I0, U8G$1.PE0@15
- new net AD5: R94.1, U$6.A1, U1.I5, U8G$1.PE1@14
- new net AD6: R47.2, U$4.A2, U1.I6, U8G$1.PE2@13
- new net AD7: R95.1, U$4.A1, U1.I7, U8G$1.PE3@12
- new net AD8: R48.2, U$3.A2, U1.I9, U8G$1.PD3@4
- new net AD9: R96.1, U$3.A1, U1.I8, U8G$1.PD2@3
- new net CAN_RX: U15.R, U8G$1.PB0@95
- new net CAN_TX: U15.D, U8G$1.PB1@96
- new net CH1: U4.COMMON_IN/OUT
- new net CH2: U1.COMMON_IN/OUT
- new net CH3: U3.COMMON_IN/OUT
- new net D0: R54.2, U$16.A2, U4.I4, U8G$1.PN5@112
- new net D1: R102.1, U$16.A1, U4.I5, U8G$1.PN4@111
- new net D10: R59.2, U$21.A2, U4.I14, U8G$1.PM1@77
- new net D11: R107.1, U$21.A1, U4.I15, U8G$1.PM2@76
- new net D12: R60.2, U$22.A2, U3.I0, U8G$1.PM3@75
- new net D13: R108.1, U$22.A1, U3.I1, U8G$1.PM4@74
- new net D14: R61.2, U$23.A2, U3.I2, U8G$1.PM5@73
- new net D15: R109.1, U$23.A1, U3.I3, U8G$1.PM6@72
- new net D16: R62.2, U$24.A2, U3.I4, U8G$1.PM7@71
- new net D19: R111.1, U$50.A1, U3.I7, U8G$1.PK6@61
- new net D2: R55.2, U$17.A2, U4.I6, U8G$1.PQ0@5
- new net D20: R64.2, U$49.A2, U3.I15, U8G$1.PK7@60
- new net D21: R112.1, U$49.A1, U3.I14, U8G$1.PF4@46
- new net D22: R65.2, U$37.A2, U3.I13, U8G$1.PF3@45
- new net D23: R113.1, U$37.A1, U3.I12, U8G$1.PF2@44
- new net D24: R66.2, U$36.A2, U3.I11, U8G$1.PF1@43
- new net D25: R114.1, U$36.A1, U3.I10, U8G$1.PF0@42
- new net D26: U3.I9
- new net D27: U3.I8
- new net D3: R103.1, U$17.A1, U4.I7, U8G$1.PQ1@6
- new net D4: R56.2, U$18.A2, U4.I8, U8G$1.PQ4@102
- new net D5: R104.1, U$18.A1, U4.I9, U8G$1.PL3@84
- new net D6: R57.2, U$19.A2, U4.I10, U8G$1.PL2@83
- new net D7: R105.1, U$19.A1, U4.I11, U8G$1.PL1@82
- new net D8: R58.2, U$20.A2, U4.I12, U8G$1.PL0@81
- new net D9: R106.1, U$20.A1, U4.I13, U8G$1.PM0@78
- new net DUT_AOUT1: JP3.12, R82.2, U$45.A2, U5.VOUT
- new net DUT_CAN_N: JP11.1, JP3.2, R87.2, U$25.A2, U15.CANL
- new net DUT_CAN_P: JP3.1, R135.1, R140.2, U$25.A1, U15.CANH
- new net DUT_CS: JP3.6, JP4.1, JP7.1, R85.2, U$48.A2, U8G$1.PA3@36
- new net DUT_LIN: JP3.13, JP9.2, R129.1, U$44.A1, U7.LBUS
- new net DUT_MISO: JP3.4, R86.2, U$26.A2, U8G$1.PA2@35
- new net DUT_MOSI: JP3.7, R132.1, U$47.A1, U8G$1.PA4@37
- new net DUT_ONEWIRE: JP3.3, R134.1, U$26.A1, U8G$1.PQ2@11
- new net DUT_RX: JP3.10, R83.2, U$46.A2, U8G$1.PA0@33
- new net DUT_SCL: JP3.8, R131.1, R80.2, U$46.A1, U8G$1.PB2@91
- new net DUT_SCLK: JP3.5, R133.1, U$48.A1, U8G$1.PA5@38
- new net DUT_SDA: JP3.9, R81.2, R84.2, U$47.A2, U8G$1.PB3@92
- new net DUT_SH-: R17.1, R39.2, U$9.A2, U12.VIN-
- new net DUT_TX: JP3.11, R130.1, U$45.A1, U8G$1.PA1@34
- new net LIN_CS: U7.CS, U8G$1.PC5@24
- new net LIN_RX: U7.RXD, U8G$1.PA6@40
- new net LIN_TX: U7.TXD, U8G$1.PA7@41
- new net M0OUT: X4.1
- new net N$153: LED10.A, R40.1
- new net PC4: U8G$1.PC4@25
- new net POWER_IN_12V: C25.1, C26.1, C5.1, D1.A, R118.2, R40.2, S1.O, U16.IN, U2.IN, U6.IN, U7.VBB
- new net SW1: S3.3, U8G$1.PH0@29
- new net SW2: S3.2, U8G$1.PG0@49
- new net SW3: S3.1, U8G$1.PG1@50
- new net SWO/TDO/MOSI: ISP1.MISO, J1.TDO, JP2.13, R12.1, SV1.15
- new net TSTR_SCL1: JP4.2, R78.1
- net !RESET: now also JP1.2; no longer S2.1@A, S2.1@B
- net DUT_CONNECT: now also U8G$1.PL4@85
- net DUT_SH+: now also R91.1, U$9.A1
- net GND: now also JP13.P$1, JP6.58, JP6.60, LED10.C, R115.1, R119.1, R136.2, R139.2, R36.2, R46.2, R68.2, R74.1, R76.1, R77.2, R79.2, U15.GND, U5.VSS, U7.VSS; no longer C11.2, C6.2, IC1.VSS, R44.1, R46.1, S2.0@A, S2.0@B, U$10.C, U$11.C, U$12.C, U$27.C, U$28.C, U$29.C, U$30.C, U$31.C, U$32.C, U$33.C, U$35.C, U$38.C, U$39.C, U$40.C, U$41.C, U$42.C, U$43.C, U10.A0, U11.A1, U12.A0, U12.A1, U5.GND, U5.~E, X3.2
- net HOST_GND: now also C6.2, C7.2, JP8.GND, U$10.C, U$5.C, U17.GND, U17.GND_2; no longer C39.1, C45.1, C49.1, U13.GND, U13.GND@1
- net HOST_UART_RX: now also U17.RXD; no longer U13.RXD
- net HOST_UART_TX: now also U17.TXD; no longer U13.TXD
- net LDO1: now also JP6.5, JP6.59, JP6.6; no longer R108.1, R29.2, R60.2, U$22.A1, U$22.A2
- net LDO1_ENABLE: now also U8G$1.PH3@32
- net LDO1_SH+: now also R29.2
- net LDO2: now also JP6.3, JP6.4; no longer R109.1, R30.2, R61.2, U$23.A1, U$23.A2
- net LDO2_ENABLE: now also U8G$1.PH2@31
- net LDO2_SH+: now also R30.2
- net LDO3: now also JP6.1, JP6.2; no longer R110.1, R33.2, R62.2, U$24.A1, U$24.A2
- net LDO3_ENABLE: now also U8G$1.PH1@30
- net LDO3_SH+: now also R33.2
- net M0S0: now also U4.S3, U8G$1.PN0@107; no longer U4.S0
- net M0S1: now also U4.S2, U8G$1.PN1@108; no longer U4.S1
- net M0S2: now also U4.S1, U8G$1.PN2@109; no longer U4.S2
- net M0S3: now also U4.S0, U8G$1.PN3@110; no longer U4.S3
- net M1OUT: no longer U1.COMMON_IN/OUT, U4.COMMON_IN/OUT
- net M1S0: now also U8G$1.PJ0@116
- net M1S1: now also U8G$1.PJ1@117
- net M1S2: now also U8G$1.PP1@119
- net M1S3: now also U8G$1.PP0@118
- net M2OUT: no longer U3.COMMON_IN/OUT, U5.COMMON_IN/OUT
- net M2S0: now also U8G$1.PP2@103
- net M2S1: now also U8G$1.PP3@104
- net M2S2: now also U8G$1.PP4@105
- net M2S3: now also U8G$1.PP5@106
- net N$1: now also R46.1, U5.A0; no longer JP3.12
- net N$112: now also R119.2, U15.RS; no longer R18.2, U$12.A2
- net N$180: no longer U$35.A2
- net N$2: now also JP11.2, R140.1; no longer R10.2, R13.2, R14.2, R15.2, R9.2
- net N$4: now also R87.1, SV1.2; no longer JP6.1, R18.1
- net N$40: now also F1.1, JP12.P$1, JP5.PWR; no longer JP6.59, R69.1
- net N$41: now also R18.1, S3.6; no longer JP7.1, R70.1
- net N$42: now also R19.1, S3.5; no longer JP7.3, R71.1
- net N$43: now also R34.1, S3.4; no longer JP7.5, R72.1
- net N$44: now also R71.1, U17.RESET; no longer JP4.2, R41.1
- net N$45: now also R73.1, U10.A1; no longer R40.2, R46.2
- net N$46: now also R75.1, U11.A0; no longer IC1.RXD, R40.1
- net N$47: now also D1.C, R117.1; no longer IC1.TXD
- net N$48: now also R74.2, U10.A0; no longer IC1.RS, R44.2
- net N$49: now also JP7.2, R79.1; no longer JP7.7, R73.1
- net N$50: now also R76.2, U11.A1; no longer JP7.9, R74.1
- net N$51: now also R77.1, U12.A0, U12.A1; no longer JP7.11, R75.1
- net N$52: now also JP10.2, R80.1, R81.1; no longer JP7.13, R76.1
- net N$58: now also SV1.12; no longer JP7.25
- net N$59: now also SV1.10; no longer JP7.27
- net N$6: now also R135.2, SV1.1; no longer JP6.3, R19.1
- net N$60: now also SV1.8; no longer JP7.29
- net N$61: now also SV1.6; no longer JP7.31
- net N$62: now also SV1.4; no longer JP7.33
- net N$64: now also R118.1, U7.!WAKE; no longer JP7.2, R118.2
- net N$65: now also JP9.1, R117.2; no longer JP7.4, R119.2
- net N$7: now also F1.2, S1.P; no longer JP6.5, R34.1
- net N$75: now also SV1.13; no longer JP7.24
- net N$76: now also SV1.11; no longer JP7.26
- net N$77: now also SV1.9; no longer JP7.28
- net N$78: now also SV1.7; no longer JP7.30
- net N$79: now also SV1.5; no longer JP7.32
- net N$80: now also SV1.3; no longer JP7.34
- net NRESET: now also R32.1, SV1.20; no longer JP1.2
- net SWDCLK/TCLK/SCK: now also R28.2, R4.1, SV1.16
- net SWDIO/TMS: now also R11.1, SV1.18
- net TDI/MISO: now also ISP1.MOSI, J1.TDI, R31.1, SV1.17
- net TEST_FAIL: now also U8G$1.PL5@86
- net TEST_PASS: now also R41.2, U8G$1.PL7@93
- net TEST_RUN: now also R44.2, U8G$1.PL6@94
- net TSTR_3V3: now also C3.1, JP10.1, JP2.1, R10.2, R11.2, R12.2, R13.2, R14.2, R15.2, R18.2, R19.2, R31.2, R32.2, R34.2, R4.2, R69.2, R70.2, R72.1, R73.2, R75.2, R78.2, R9.2, U1.VCC, U15.VCC, U3.VCC, U4.VCC, U5.VDD; no longer U10.A1, U11.A0, U9.VS
- net TSTR_RX: now also U8G$1.PC7@22; no longer JP3.10, U8G$1.PA0@33
- net TSTR_SCL: now also R110.1, R69.1, U$24.A1, U3.I5, U5.SCL, U8G$1.PK4@63
- net TSTR_SDA: now also R63.2, R70.1, U$50.A2, U3.I6, U5.SDA, U8G$1.PK5@62
- net TSTR_TX: now also U8G$1.PC6@23; no longer JP3.11, U8G$1.PA1@34
- net USBD_N: now also U17.USBDM; no longer U13.USBDM
- net USBD_P: now also U17.USBDP; no longer U13.USBDP
- net USB_N: now also R41.1, U$5.A1
- net USB_P: now also R44.1, U$5.A2
- net VBUS: now also C6.1, C7.1, R71.2, U$10.A1, U17.VCC, U17.VCCIO; no longer C45.2, C49.2, U13.VCC, U13.VCCIO
- net VCC: now also R72.2, U9.VS; no longer JP1.6, JP2.1, U3.VCC, U5.VCC
Other:
- note added: "Master mode jumper"
- note added: "east"
- note added: "north"
- note added: "north east"
- note added: "south"
- note removed: "Ethernet Activity LED"
- note removed: "Ethernet Link LED"
- note removed: "JTAG Signals"
- note removed: "Serial0 back to programmer"
