File: RelayBoard/RelayBoard.brd (EAGLE design)
At the start: 129.1 x 103.7 mm, 243 parts, among them J1 JTAG_ARM_10PIN, J4 JTAG_ARM_10PIN, U1 CD74HC4067SM96, U10 INA219AIDCNR, U11 INA219AIDCNR, U12 INA219AIDCNR, U14 ADUM1201ARZ, U15 SN65HVD230D, U16 TL1963AKTTR., U17 FT230XS, U2 TL1963AKTTR., U3 CD74HC4067SM96, U4 CD74HC4067SM96, U5 MCP4725A0T-E/CH, U6 TL1963AKTTR., U7 MCP2003-E/SN, U8 TM4C1294NCPDT, U9 INA219AIDCNR, X1 A1944-50, X2 A1944-50, X4 A1944-50, Y3 NX3225GA

Commit message: Fix issues
Parts:
- flipped R35 to the bottom
Routing:
- net ADJ3: track 20.7 -> 20.1 mm, vias 3 -> 2
- net GND: track 310.9 -> 310.4 mm, vias 79 -> 78
Changed lines of the file:
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@@
 </element>
 <element name="R2" library="resistor" package="R0402" value="" x="62.992" y="27.0764" rot="MR270"/>
-<element name="R35" library="resistor" package="R0402" value="" x="52.451" y="32.004"/>
+<element name="R35" library="resistor" package="R0402" value="" x="52.451" y="32.004" rot="MR0"/>
 <element name="R36" library="resistor" package="R0402" value="4k7" x="50.927" y="29.3878" rot="MR180"/>
 <element name="U2" library="TL1963" package="TO170P1485X457-6N" value="TL1963AKTTR." x="42.926" y="19.1008" rot="MR180">
@@
 <wire x1="42.7228" y1="29.1592" x2="42.7228" y2="30.0586" width="0.508" layer="16"/>
 <wire x1="42.7228" y1="30.0586" x2="42.7378" y2="30.0736" width="0.508" layer="16"/>
-<wire x1="51.801" y1="32.004" x2="53.101" y2="30.6278" width="0.508" layer="1"/>
+<wire x1="53.101" y1="32.004" x2="53.101" y2="30.6278" width="0.508" layer="16"/>
 <wire x1="53.101" y1="30.6278" x2="53.198" y2="30.5308" width="0.508" layer="16"/>
 <wire x1="57.15" y1="27.7114" x2="57.15" y2="28.956" width="0.508" layer="16"/>
@@
 <wire x1="53.8734" y1="25.6794" x2="57.15" y2="25.6794" width="0.254" layer="1"/>
 <contactref element="JP13" pad="P$1"/>
-<via x="53.101" y="30.6278" extent="1-16" drill="0.3048"/>
 </signal>
 <signal name="NRESET">
@@
 <contactref element="U8" pad="P$64"/>
 <contactref element="R20" pad="1"/>
-<wire x1="59.929" y1="37.3634" x2="59.7154" y2="37.3634" width="0" layer="19" extent="1-16"/>
 <via x="59.7154" y="37.3634" extent="1-16" drill="0.3048"/>
 <wire x1="59.7154" y1="37.3634" x2="60.325" y2="38.1" width="0.2286" layer="16"/>
@@
 <wire x1="62.992" y1="27.7264" x2="60.5686" y2="27.7264" width="0.254" layer="16"/>
 <wire x1="60.5686" y1="27.7264" x2="60.5536" y2="27.7114" width="0.254" layer="16"/>
-<wire x1="53.101" y1="32.004" x2="51.801" y2="30.9014" width="0.2286" layer="1"/>
+<wire x1="51.801" y1="32.004" x2="51.801" y2="30.9014" width="0.2286" layer="16"/>
 <wire x1="51.801" y1="30.9014" x2="52.07" y2="30.6324" width="0.2286" layer="16"/>
 <via x="52.07" y="30.6324" extent="1-16" drill="0.3048" diameter="0.3048"/>
@@
 <wire x1="64.0334" y1="27.6352" x2="54.8894" y2="27.6352" width="0.254" layer="1"/>
 <wire x1="54.8894" y1="27.6352" x2="53.4289" y2="29.0957" width="0.254" layer="1"/>
-<via x="51.801" y="30.9014" extent="1-16" drill="0.3048"/>
 </signal>
 <signal name="LDO1_ENABLE">
