File: HIL/RACK.brd (EAGLE design)
At the start: 523 x 690.4 mm, 0 parts

Commit message: Generate pdfs, and gerbers Libraries “>NAME” parameter change
Other:
- board size 523 x 690.4 mm -> 442.9 x 510.1 mm
- board text added: "Display"
- board text added: "FRONT"
- board text added: "TOP"
Changed lines of the file:
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@@
 <board>
 <plain>
-<wire x1="0" y1="0" x2="439.7968" y2="0" width="0.254" layer="20"/>
-<wire x1="439.7968" y1="0" x2="439.7968" y2="150.0762" width="0.254" layer="20"/>
-<wire x1="439.7968" y1="150.0762" x2="0" y2="88" width="0.254" layer="20"/>
-<wire x1="0" y1="88" x2="0" y2="0" width="0.254" layer="20"/>
-<wire x1="83.0326" y1="408.3558" x2="523.0326" y2="408.3558" width="0.254" layer="20"/>
-<wire x1="523.0326" y1="408.3558" x2="523.0326" y2="690.3558" width="0.254" layer="20"/>
-<wire x1="523.0326" y1="690.3558" x2="83.0326" y2="690.3558" width="0.254" layer="20"/>
-<wire x1="83.0326" y1="690.3558" x2="83.0326" y2="408.3558" width="0.254" layer="20"/>
-<wire x1="375.4628" y1="534.9458" x2="375.4628" y2="429.9458" width="0.254" layer="20"/>
-<wire x1="375.4628" y1="429.9458" x2="505.4628" y2="429.9458" width="0.254" layer="20"/>
-<wire x1="505.4628" y1="429.9458" x2="505.4628" y2="534.9458" width="0.254" layer="20"/>
-<wire x1="505.4628" y1="534.9458" x2="375.4628" y2="534.9458" width="0.254" layer="20"/>
-<text x="405.257" y="497.2558" size="6.4516" layer="20">HILTester</text>
-<wire x1="95.7542" y1="434.9496" x2="154.2542" y2="434.9496" width="0.254" layer="20"/>
-<wire x1="154.2542" y1="434.9496" x2="154.2542" y2="522.0496" width="0.254" layer="20"/>
-<wire x1="154.2542" y1="522.0496" x2="95.7542" y2="522.0496" width="0.254" layer="20"/>
-<wire x1="95.7542" y1="522.0496" x2="95.7542" y2="434.9496" width="0.254" layer="20"/>
-<text x="117.221" y="452.8566" size="6.4516" layer="20" rot="R90">RPI</text>
-<wire x1="96.4438" y1="575.437" x2="147.2438" y2="575.437" width="0.254" layer="20"/>
-<wire x1="147.2438" y1="575.437" x2="147.2438" y2="677.037" width="0.254" layer="20"/>
-<wire x1="147.2438" y1="677.037" x2="96.4438" y2="677.037" width="0.254" layer="20"/>
-<wire x1="96.4438" y1="677.037" x2="96.4438" y2="575.437" width="0.254" layer="20"/>
-<text x="110.109" y="593.4202" size="6.4516" layer="20" rot="R90">PSU</text>
-<wire x1="374.8278" y1="657.1198" x2="374.8278" y2="552.1198" width="0.254" layer="20"/>
-<wire x1="374.8278" y1="552.1198" x2="504.8278" y2="552.1198" width="0.254" layer="20"/>
-<wire x1="504.8278" y1="552.1198" x2="504.8278" y2="657.1198" width="0.254" layer="20"/>
-<wire x1="504.8278" y1="657.1198" x2="374.8278" y2="657.1198" width="0.254" layer="20"/>
-<text x="404.622" y="619.4298" size="6.4516" layer="20">HILTester</text>
-<wire x1="225.2472" y1="534.9458" x2="225.2472" y2="429.9458" width="0.254" layer="20"/>
-<wire x1="225.2472" y1="429.9458" x2="355.2472" y2="429.9458" width="0.254" layer="20"/>
-<wire x1="355.2472" y1="429.9458" x2="355.2472" y2="534.9458" width="0.254" layer="20"/>
-<wire x1="355.2472" y1="534.9458" x2="225.2472" y2="534.9458" width="0.254" layer="20"/>
-<text x="255.0414" y="497.2558" size="6.4516" layer="20">HILTester</text>
-<wire x1="224.6122" y1="657.1198" x2="224.6122" y2="552.1198" width="0.254" layer="20"/>
-<wire x1="224.6122" y1="552.1198" x2="354.6122" y2="552.1198" width="0.254" layer="20"/>
-<wire x1="354.6122" y1="552.1198" x2="354.6122" y2="657.1198" width="0.254" layer="20"/>
-<wire x1="354.6122" y1="657.1198" x2="224.6122" y2="657.1198" width="0.254" layer="20"/>
-<text x="254.4064" y="619.4298" size="6.4516" layer="20">HILTester</text>
+<wire x1="9.9314" y1="205.4098" x2="449.9314" y2="205.4098" width="0.254" layer="20"/>
+<wire x1="449.9314" y1="205.4098" x2="449.9314" y2="293.4098" width="0.254" layer="20"/>
+<wire x1="449.9314" y1="293.4098" x2="9.9314" y2="293.4098" width="0.254" layer="20"/>
+<wire x1="9.9314" y1="293.4098" x2="9.9314" y2="205.4098" width="0.254" layer="20"/>
+<wire x1="11.8872" y1="433.5018" x2="451.8872" y2="433.5018" width="0.254" layer="20"/>
+<wire x1="451.8872" y1="433.5018" x2="451.8872" y2="715.5018" width="0.254" layer="20"/>
+<wire x1="451.8872" y1="715.5018" x2="11.8872" y2="715.5018" width="0.254" layer="20"/>
+<wire x1="11.8872" y1="715.5018" x2="11.8872" y2="433.5018" width="0.254" layer="20"/>
+<wire x1="304.3174" y1="560.0918" x2="304.3174" y2="455.0918" width="0.254" layer="20"/>
+<wire x1="304.3174" y1="455.0918" x2="434.3174" y2="455.0918" width="0.254" layer="20"/>
+<wire x1="434.3174" y1="455.0918" x2="434.3174" y2="560.0918" width="0.254" layer="20"/>
+<wire x1="434.3174" y1="560.0918" x2="304.3174" y2="560.0918" width="0.254" layer="20"/>
+<text x="334.1116" y="522.4018" size="6.4516" layer="20">HILTester</text>
+<wire x1="24.6088" y1="460.0956" x2="83.1088" y2="460.0956" width="0.254" layer="20"/>
+<wire x1="83.1088" y1="460.0956" x2="83.1088" y2="547.1956" width="0.254" layer="20"/>
+<wire x1="83.1088" y1="547.1956" x2="24.6088" y2="547.1956" width="0.254" layer="20"/>
+<wire x1="24.6088" y1="547.1956" x2="24.6088" y2="460.0956" width="0.254" layer="20"/>
+<text x="46.0756" y="478.0026" size="6.4516" layer="20" rot="R90">RPI</text>
+<wire x1="25.2984" y1="600.583" x2="76.0984" y2="600.583" width="0.254" layer="20"/>
+<wire x1="76.0984" y1="600.583" x2="76.0984" y2="702.183" width="0.254" layer="20"/>
+<wire x1="76.0984" y1="702.183" x2="25.2984" y2="702.183" width="0.254" layer="20"/>
+<wire x1="25.2984" y1="702.183" x2="25.2984" y2="600.583" width="0.254" layer="20"/>
+<text x="38.9636" y="618.5662" size="6.4516" layer="20" rot="R90">PSU</text>
+<wire x1="303.6824" y1="682.2658" x2="303.6824" y2="577.2658" width="0.254" layer="20"/>
+<wire x1="303.6824" y1="577.2658" x2="433.6824" y2="577.2658" width="0.254" layer="20"/>
+<wire x1="433.6824" y1="577.2658" x2="433.6824" y2="682.2658" width="0.254" layer="20"/>
+<wire x1="433.6824" y1="682.2658" x2="303.6824" y2="682.2658" width="0.254" layer="20"/>
+<text x="333.4766" y="644.5758" size="6.4516" layer="20">HILTester</text>
+<wire x1="154.1018" y1="560.0918" x2="154.1018" y2="455.0918" width="0.254" layer="20"/>
+<wire x1="154.1018" y1="455.0918" x2="284.1018" y2="455.0918" width="0.254" layer="20"/>
+<wire x1="284.1018" y1="455.0918" x2="284.1018" y2="560.0918" width="0.254" layer="20"/>
+<wire x1="284.1018" y1="560.0918" x2="154.1018" y2="560.0918" width="0.254" layer="20"/>
+<text x="183.896" y="522.4018" size="6.4516" layer="20">HILTester</text>
+<wire x1="153.4668" y1="682.2658" x2="153.4668" y2="577.2658" width="0.254" layer="20"/>
+<wire x1="153.4668" y1="577.2658" x2="283.4668" y2="577.2658" width="0.254" layer="20"/>
+<wire x1="283.4668" y1="577.2658" x2="283.4668" y2="682.2658" width="0.254" layer="20"/>
+<wire x1="283.4668" y1="682.2658" x2="153.4668" y2="682.2658" width="0.254" layer="20"/>
+<text x="183.261" y="644.5758" size="6.4516" layer="20">HILTester</text>
+<text x="11.5062" y="295.1988" size="6.4516" layer="20">FRONT</text>
+<text x="14.9606" y="717.6516" size="6.4516" layer="20">TOP</text>
+<wire x1="8.9916" y1="316.6364" x2="448.9916" y2="316.6364" width="0.254" layer="20"/>
+<wire x1="448.9916" y1="316.6364" x2="448.9916" y2="404.6364" width="0.254" layer="20"/>
+<wire x1="448.9916" y1="404.6364" x2="8.9916" y2="404.6364" width="0.254" layer="20"/>
+<wire x1="8.9916" y1="404.6364" x2="8.9916" y2="316.6364" width="0.254" layer="20"/>
+<text x="10.5664" y="406.4254" size="6.4516" layer="20">FRONT</text>
+<wire x1="192.3288" y1="231.8766" x2="192.3288" y2="271.8766" width="0.254" layer="20"/>
+<wire x1="192.3288" y1="271.8766" x2="252.3288" y2="271.8766" width="0.254" layer="20"/>
+<wire x1="252.3288" y1="271.8766" x2="252.3288" y2="231.8766" width="0.254" layer="20"/>
+<wire x1="252.3288" y1="231.8766" x2="192.3288" y2="231.8766" width="0.254" layer="20"/>
+<text x="209.7024" y="251.8664" size="6.4516" layer="20">Display</text>
 </plain>
 <attributes>
