File: HIL/HIL.brd (EAGLE design)
At the start: 129.6 x 111 mm, 295 parts, among them J1 JTAG_ARM_10PIN, J4 JTAG_ARM_10PIN, M0S0 TPB1,27, M0S1 TPB1,27, M0S2 TPB1,27, M0S3 TPB1,27, M1S0 M0S3, M1S1 M0S3, M1S2 M0S3, M1S3 M0S3, M2S0 M0S3, M2S1 M0S3, M2S2 M0S3, M2S3 M0S3, SW1 EC12E_SW, U1 CD74HC4067SM96, U10 INA219AIDCNR, U11 INA219AIDCNR, U12 INA219AIDCNR, U13 TM4C1294NCPDT, U14 ADUM1201ARZ, U15 SN65HVD230D, U16 TL1963AKTTR., U17 FT230XS, U2 TL1963AKTTR., U3 CD74HC4067SM96, U4 CD74HC4067SM96, U5 MAX11647EUA+T, U6 TL1963AKTTR., U7 MCP2003-E/SN, U8 DAC7578SPW, U9 INA219AIDCNR, X1 A1944-50, X2 A1944-50, X4 A1944-50, Y3 NX3225GA

Commit message: start the A3.0
Parts:
- removed C13, C14, C16, C17, C18, C19, C20, C6: 0.1uF, rcl:C0402K
- removed C15: 2.2uF, rcl:C0402K
- removed C36, C9: 12pF, rcl:C0402K
- removed C37: 0.1uF, eagle-ltspice:C0402
- removed C7: 10uF, rcl:C0402K
- removed JP1: RESET, SparkFun-Retired:SJ_2S-NO
- removed JP14, JP15: (no value), JDT-1800_smahed:1X03-CLEANBIG
- removed R18, R19, R71: 4.7k, resistor:R0402
- removed R20: 1M, rcl:R0402
- removed R21: 51, rcl:R0402
- removed R22: 4.87k 1%, rcl:R0402
- removed R23: 2k, rcl:R0402
- removed R24: 100, rcl:R0402
- removed R25: 10k, rcl:R0402
- removed SW1: EC12E_SW, switch-alps:ALPS_EC12E_SW
- removed U13: TM4C1294NCPDT, ti-tiva:TQFP128
- removed U14: ADUM1201ARZ, ADUM1201ARZ:SOIC127P600X175-8N
- removed U17: FT230XS, FT230XS:SOP63P600X175-16N
- removed X4: A1944-50, con-coax:A1944
- removed Y3: NX3225GA, MRDT-Passives:NDK3.2X2.5
- added JP19: (no value), JDT-1800_smahed:2X04
- added JP20: (no value), pinhead:2X30
- added SV2: (no value), con-lstb:MA10-2
- added U$30: STM32F4-DISCOVERY_STM32F4-DISCOVERY, stm32f4-discovery-breakout-v1:STM32F4-DISCOVERY_STM32F4-DISCOVERY
- added X3: BU-SMA-V, con-coax:BU-SMA-V
- F1: value (none) -> PTCSMD-W; device fuse:GSH15 -> SparkFun-PowerIC:PTC-1206-WIDE
- X1, X2: value A1944-50 -> BU-SMA-V; device con-coax:A1944 -> con-coax:BU-SMA-V
- moved R10 97.7 mm to (-24.6, 19.5)
- moved R13 97.7 mm to (-32.3, 4.75), flipped to the top
- moved R15 97.7 mm to (-29.4, 8.94), flipped to the top
- moved R9 97.7 mm to (-31.0, 4.72), flipped to the top
- moved J4 97.7 mm to (-36.4, 7.09), flipped to the top
- moved R14 97.7 mm to (-33.9, 4.75), flipped to the top
- moved X2 14.7 mm to (119.8, 42.7), turned to 90 degrees
- moved X1 13.4 mm to (119.8, 27.8), turned to 90 degrees
- moved F1 7.41 mm to (21.9, 24.3), turned to 270 degrees
- moved JP3 3.27 mm to (127.4, 82.0)
Connections:
- removed net HOST_UART_RX: U14.6, U17.4
- removed net HOST_UART_TX: U14.7, U17.1
- removed net N$44: R71.1, U17.11
- removed net N$82: R19.1, SW1.C
- removed net N_$2: C20.1, C37.1, R20.1, R21.1, R24.1, R25.2, U13.64, U13.68, U13.70
- removed net N_$28: C13.1, C14.1, C15.1, U13.115, U13.87
- removed net N_$29: R22.2, U13.59
- removed net N_$30: R23.2, U13.89
- removed net N_$31: C36.1, U13.88, Y3.P$3
- removed net N_$32: C9.1, R23.1, Y3.P$1
- removed net PC4: U13.25
- removed net ROTARY_A: SW1.A, U13.49
- removed net ROTARY_B: SW1.B, U13.50
- removed net ROTARY_SW: SW1.D, U13.29
- removed net VBUS: C6.1, C7.1, JP8.VBUS, R71.2, U$10.1, U14.8, U17.12, U17.3
- new net N$67: SV1.19, SV2.19
- new net N$73: JP8.VBUS, U$10.1
- net !RESET: no longer JP1.2, R24.2
- net AD0: no longer U13.21
- net AD1: no longer U13.20
- net AD10: no longer U13.2
- net AD11: no longer U13.1
- net AD12: no longer U13.128
- net AD13: no longer U13.127
- net AD14: no longer U13.126
- net AD15: no longer U13.125
- net AD16: no longer U13.124
- net AD17: no longer U13.123
- net AD18: no longer U13.121
- net AD19: no longer U13.120
- net AD2: no longer U13.19
- net AD3: no longer U13.18
- net AD4: no longer U13.15
- net AD5: no longer U13.14
- net AD6: no longer U13.13
- net AD7: no longer U13.12
- net AD8: no longer U13.4
- net AD9: no longer U13.3
- net AOUT_1: now also JP19.1
- net AOUT_2: now also JP19.2
- net AOUT_3: now also JP19.3
- net AOUT_4: now also JP19.4
- net AOUT_5: now also JP19.5
- net AOUT_6: now also JP19.6
- net AOUT_7: now also JP19.7
- net AOUT_8: now also JP19.8
- net CAN_RX: no longer U13.95
- net CAN_TX: no longer U13.96
- net CH1: now also X1.1; no longer X2.1
- net CH2: now also X2.1; no longer X1.1
- net CH3: now also X3.1; no longer X4.1
- net D0: no longer U13.112
- net D1: no longer U13.111
- net D10: no longer U13.77
- net D11: no longer U13.76
- net D12: no longer U13.75
- net D13: no longer U13.74
- net D14: no longer U13.73
- net D15: no longer U13.72
- net D16: no longer U13.71
- net D19: no longer U13.61
- net D2: no longer U13.5
- net D20: no longer U13.60
- net D21: no longer U13.46
- net D22: no longer U13.45
- net D23: no longer U13.44
- net D24: no longer U13.43
- net D25: no longer U13.42
- net D3: no longer U13.6
- net D4: no longer U13.102
- net D5: no longer U13.84
- net D6: no longer U13.83
- net D7: no longer U13.82
- net D8: no longer U13.81
- net D9: no longer U13.78
- net DUT_CONNECT: no longer U13.85
- net DUT_CS: no longer U13.36
- net DUT_MISO: no longer U13.35
- net DUT_MOSI: no longer U13.37
- net DUT_ONEWIRE: no longer U13.11
- net DUT_RX: no longer U13.33
- net DUT_SCL: no longer U13.91
- net DUT_SCLK: no longer U13.38
- net DUT_SDA: no longer U13.92
- net DUT_TX: no longer U13.34
- net GND: now also JP20.58, JP20.60, X3.2, X3.3, X3.4, X3.5; no longer C13.2, C14.2, C15.2, C16.2, C17.2, C18.2, C19.2, C20.2, C36.2, C37.2, C9.2, JP1.1, JP14.1, JP15.1, R22.1, SW1.GND1, SW1.GND2, U13.10, U13.114, U13.17, U13.48, U13.55, U13.58, U13.80, U14.4, X4.2, X4.3, X4.4, X4.5
- net HOST_GND: no longer C6.2, C7.2, U14.5, U17.13, U17.5
- net LDO1: now also JP20.5, JP20.59, JP20.6
- net LDO1_ENABLE: no longer U13.32
- net LDO2: now also JP20.3, JP20.4
- net LDO2_ENABLE: no longer U13.31
- net LDO3: now also JP20.1, JP20.2
- net LDO3_ENABLE: no longer U13.30
- net LIN_CS: no longer U13.24
- net LIN_RX: no longer U13.40
- net LIN_TX: no longer U13.41
- net M0S0: no longer U13.107
- net M0S1: no longer U13.108
- net M0S2: no longer U13.109
- net M0S3: no longer U13.110
- net M1S0: no longer U13.116
- net M1S1: no longer U13.117
- net M1S2: no longer U13.119
- net M1S3: no longer U13.118
- net M2S0: no longer U13.103
- net M2S1: no longer U13.104
- net M2S2: no longer U13.105
- net M2S3: no longer U13.106
- net N$10: now also JP20.11
- net N$100: now also JP20.38
- net N$101: now also JP20.40
- net N$102: now also JP20.42
- net N$103: now also JP20.44
- net N$104: now also JP20.46
- net N$105: now also JP20.48
- net N$106: now also JP20.50
- net N$107: now also JP20.52
- net N$108: now also JP20.54
- net N$109: now also JP20.56
- net N$11: now also JP20.13
- net N$12: now also JP20.15
- net N$13: now also JP20.17
- net N$14: now also JP20.19
- net N$15: now also JP20.21
- net N$16: now also JP20.23
- net N$17: now also JP20.25
- net N$18: now also JP20.27
- net N$19: now also JP20.29
- net N$20: now also JP20.31
- net N$21: now also JP20.33
- net N$22: now also JP20.35
- net N$24: now also JP20.37
- net N$26: now also JP20.39
- net N$27: now also JP20.41
- net N$28: now also JP20.43
- net N$29: now also JP20.45
- net N$30: now also JP20.47
- net N$31: now also JP20.49
- net N$32: now also JP20.51
- net N$37: now also JP20.53
- net N$38: now also JP20.55
- net N$39: now also JP20.57
- net N$4: now also SV2.2
- net N$43: now also SV1.14, SV2.14; no longer R18.1, SW1.E
- net N$58: now also SV2.12
- net N$59: now also SV2.10
- net N$6: now also SV2.1
- net N$60: now also SV2.8
- net N$61: now also SV2.6
- net N$62: now also SV2.4
- net N$7: now also F1.1; no longer F1.2
- net N$75: now also SV2.13
- net N$76: now also SV2.11
- net N$77: now also SV2.9
- net N$78: now also SV2.7
- net N$79: now also SV2.5
- net N$8: now also JP20.7
- net N$80: now also SV2.3
- net N$85: now also JP20.8
- net N$86: now also JP20.10
- net N$87: now also JP20.12
- net N$88: now also JP20.14
- net N$89: now also JP20.16
- net N$9: now also JP20.9
- net N$90: now also JP20.18
- net N$91: now also JP20.20
- net N$92: now also JP20.22
- net N$93: now also JP20.24
- net N$94: now also JP20.26
- net N$95: now also JP20.28
- net N$96: now also JP20.30
- net N$97: now also JP20.32
- net N$98: now also JP20.34
- net N$99: now also JP20.36
- net NRESET: now also SV2.20
- net SWDCLK/TCLK/SCK: now also SV2.16
- net SWDIO/TMS: now also SV2.18
- net SWO/TDO/MOSI: now also SV2.15
- net TARGET_TCK/SWCLK: no longer U13.100
- net TARGET_TDI: no longer U13.98
- net TARGET_TDO/SWO: no longer U13.97
- net TARGET_TMS/SWDIO: no longer U13.99
- net TDI/MISO: now also SV2.17
- net TEST_FAIL: no longer U13.86
- net TEST_PASS: no longer U13.93
- net TEST_RUN: no longer U13.94
- net TSTR_3V3: no longer C16.1, C17.1, C18.1, C19.1, R18.2, R19.2, R20.2, R21.2, R25.1, U13.101, U13.113, U13.122, U13.16, U13.26, U13.28, U13.39, U13.47, U13.51, U13.52, U13.69, U13.7, U13.79, U13.8, U13.9, U13.90, U14.1
- net TSTR_RX: no longer JP14.3, JP15.3, U13.22, U14.2
- net TSTR_SCL: no longer U13.63
- net TSTR_SDA: no longer U13.62
- net TSTR_TX: no longer JP14.2, JP15.2, U13.23, U14.3
- net USBD_N: no longer U17.9
- net USBD_P: no longer U17.8
- net VIN: now also F1.2; no longer F1.1
Routing:
- net TSTR_3V3: track 311.0 -> 109.7 mm, vias 69 -> 35
- net DUT_MISO: track 143.9 -> 22.4 mm
- net CH2: track 119.4 -> 1.87 mm, vias 3 -> 1
- net CH1: track 111.1 -> 0.00 mm, vias 3 -> 0
- net DUT_CS: track 149.0 -> 38.8 mm
- net DUT_RX: track 143.5 -> 36.3 mm
- net TSTR_TX: track 105.2 -> 0.00 mm, vias 5 -> 0
- net CH3: track 102.4 -> 2.30 mm, vias 1 -> 0
- net TSTR_RX: track 99.5 -> 0.00 mm, vias 3 -> 0
- net TSTR_SCL: track 210.5 -> 111.6 mm, vias 7 -> 5
- net DUT_TX: track 137.7 -> 38.9 mm
- net TSTR_SDA: track 210.6 -> 112.3 mm, vias 5 -> 3
- net DUT_MOSI: track 135.0 -> 46.2 mm
- net GND: track 344.4 -> 255.9 mm, vias 84 -> 66
- net DUT_SCLK: track 129.4 -> 41.4 mm
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Other:
- board size 129.6 x 111 mm -> 129.5 x 111 mm
- board text added: "DAC out"
- board text added: "HILTester A3.0"
- board text removed: "HILTester A2.1"
- board text removed: "TSTR_UART"
