File: HIL/HIL.sch (EAGLE design)
At the start: 293 parts, among them J1 JTAG_ARM_10PIN, J4 JTAG_ARM_10PIN, M0S0 TPB1,27, M0S1 TPB1,27, M0S2 TPB1,27, M0S3 TPB1,27, M1S0 M0S3, M1S1 M0S3, M1S2 M0S3, M1S3 M0S3, M2S0 M0S3, M2S1 M0S3, M2S2 M0S3, M2S3 M0S3, SW1 EC12E_SW, U1 CD74HC4067SM96, U10 INA219AIDCNR, U11 INA219AIDCNR, U12 INA219AIDCNR, U13 TM4C1294NCPDT, U14 ADUM1201ARZ, U15 SN65HVD230D, U16 TL1963AKTTR., U17 FT230XS, U2 TL1963AKTTR., U3 CD74HC4067SM96, U4 CD74HC4067SM96, U5 MAX11647EUA+T, U6 TL1963AKTTR., U7 MCP2003-E/SN, U8 DAC7578SPW, U9 INA219AIDCNR, X1 A1944-50, X2 A1944-50, X4 A1944-50, Y3 NX3225GA

Commit message: start the A3.0
Parts:
- removed C13, C14, C16, C17, C18, C19, C20, C6: 0.1uF, rcl:C-EUC0402K
- removed C15: 2.2uF, rcl:C-EUC0402K
- removed C36, C9: 12pF, rcl:C-EUC0402K
- removed C37: 0.1uF, eagle-ltspice:CC0402
- removed C7: 10uF, rcl:C-EUC0402K
- removed JP1: RESET, SparkFun-Retired:JUMPER-2SMD-NO
- removed JP14, JP15: (no value), JDT-1800_smahed:PINHD-1X3CB
- removed R18, R19, R71: 4.7k, resistor:R-EU_R0402
- removed R20: 1M, rcl:R-EU_R0402
- removed R21: 51, rcl:R-EU_R0402
- removed R22: 4.87k 1%, rcl:R-EU_R0402
- removed R23: 2k, rcl:R-EU_R0402
- removed R24: 100, rcl:R-EU_R0402
- removed R25: 10k, rcl:R-EU_R0402
- removed SW1: EC12E_SW, switch-alps:EC12E_SW
- removed U13: TM4C1294NCPDT, ti-tiva:TM4C1294NCPDT
- removed U14: ADUM1201ARZ, ADUM1201ARZ:ADUM1201ARZ
- removed U17: FT230XS, FT230XS:FT230XS
- removed X4: A1944-50, con-coax:A1944-50
- removed Y3: NX3225GA, MRDT-Passives:NX3225GA
- added JP19: (no value), JDT-1800_smahed:PINHD-2X4
- added JP20: (no value), pinhead:PINHD-2X30
- added SV2: (no value), con-lstb:MA10-2
- added U$30: STM32F4-DISCOVERY_STM32F4-DISCOVERY, stm32f4-discovery-breakout-v1:STM32F4-DISCOVERY_STM32F4-DISCOVERY
- added X3: BU-SMA-V, con-coax:BU-SMA-V
- F1: value (none) -> PTCSMD-W; device fuse:GSH15 -> SparkFun-PowerIC:PTCSMD-W
- X1, X2: value A1944-50 -> BU-SMA-V; device con-coax:A1944-50 -> con-coax:BU-SMA-V
Connections:
- removed net HOST_UART_RX: U14.VOB, U17.RXD
- removed net HOST_UART_TX: U14.VIA, U17.TXD
- removed net N$44: R71.1, U17.RESET
- removed net N$82: R19.1, SW1G$1.C
- removed net N_$2: C20.1, C37.1, R20.1, R21.1, R24.1, R25.2, U13-PWR.!RESET@70, U13-PWR.!WAKE@64, U13-PWR.VBAT@68
- removed net N_$28: C13.1, C14.1, C15.1, U13-PWR.VDDC@115, U13-PWR.VDDC@87
- removed net N_$29: R22.2, U13-PWR.RBIAS@59
- removed net N_$30: R23.2, U13-PWR.OSC1@89
- removed net N_$31: C36.1, U13-PWR.OSC0@88, Y3.OSC1
- removed net N_$32: C9.1, R23.1, Y3.OSC0
- removed net PC4: U13-IO.PC4@25
- removed net ROTARY_A: SW1G$1.A, U13-IO.PG0@49
- removed net ROTARY_B: SW1G$1.B, U13-IO.PG1@50
- removed net ROTARY_SW: SW1G$2.1, U13-IO.PH0@29
- removed net VBUS: C6.1, C7.1, JP8.VBUS, R71.2, U$10.A1, U14.VDD2, U17.VCC, U17.VCCIO
- new net N$67: SV1.19, SV2.19
- new net N$73: JP8.VBUS, U$10.A1
- net !RESET: no longer JP1.2, R24.2
- net AD0: no longer U13-IO.PK3@21
- net AD1: no longer U13-IO.PK2@20
- net AD10: no longer U13-IO.PD1@2
- net AD11: no longer U13-IO.PD0@1
- net AD12: no longer U13-IO.PD7@128
- net AD13: no longer U13-IO.PD6@127
- net AD14: no longer U13-IO.PD5@126
- net AD15: no longer U13-IO.PD4@125
- net AD16: no longer U13-IO.PE5@124
- net AD17: no longer U13-IO.PE4@123
- net AD18: no longer U13-IO.PB4@121
- net AD19: no longer U13-IO.PB5@120
- net AD2: no longer U13-IO.PK1@19
- net AD3: no longer U13-IO.PK0@18
- net AD4: no longer U13-IO.PE0@15
- net AD5: no longer U13-IO.PE1@14
- net AD6: no longer U13-IO.PE2@13
- net AD7: no longer U13-IO.PE3@12
- net AD8: no longer U13-IO.PD3@4
- net AD9: no longer U13-IO.PD2@3
- net AOUT_1: now also JP19.1
- net AOUT_2: now also JP19.2
- net AOUT_3: now also JP19.3
- net AOUT_4: now also JP19.4
- net AOUT_5: now also JP19.5
- net AOUT_6: now also JP19.6
- net AOUT_7: now also JP19.7
- net AOUT_8: now also JP19.8
- net CAN_RX: no longer U13-IO.PB0@95
- net CAN_TX: no longer U13-IO.PB1@96
- net CH1: now also X1.1; no longer X2.1
- net CH2: now also X2.1; no longer X1.1
- net CH3: now also X3.1; no longer X4.1
- net D0: no longer U13-IO.PN5@112
- net D1: no longer U13-IO.PN4@111
- net D10: no longer U13-IO.PM1@77
- net D11: no longer U13-IO.PM2@76
- net D12: no longer U13-IO.PM3@75
- net D13: no longer U13-IO.PM4@74
- net D14: no longer U13-IO.PM5@73
- net D15: no longer U13-IO.PM6@72
- net D16: no longer U13-IO.PM7@71
- net D19: no longer U13-IO.PK6@61
- net D2: no longer U13-IO.PQ0@5
- net D20: no longer U13-IO.PK7@60
- net D21: no longer U13-IO.PF4@46
- net D22: no longer U13-IO.PF3@45
- net D23: no longer U13-IO.PF2@44
- net D24: no longer U13-IO.PF1@43
- net D25: no longer U13-IO.PF0@42
- net D3: no longer U13-IO.PQ1@6
- net D4: no longer U13-IO.PQ4@102
- net D5: no longer U13-IO.PL3@84
- net D6: no longer U13-IO.PL2@83
- net D7: no longer U13-IO.PL1@82
- net D8: no longer U13-IO.PL0@81
- net D9: no longer U13-IO.PM0@78
- net DUT_CONNECT: no longer U13-IO.PL4@85
- net DUT_CS: no longer U13-IO.PA3@36
- net DUT_MISO: no longer U13-IO.PA2@35
- net DUT_MOSI: no longer U13-IO.PA4@37
- net DUT_ONEWIRE: no longer U13-IO.PQ2@11
- net DUT_RX: no longer U13-IO.PA0@33
- net DUT_SCL: no longer U13-IO.PB2@91
- net DUT_SCLK: no longer U13-IO.PA5@38
- net DUT_SDA: no longer U13-IO.PB3@92
- net DUT_TX: no longer U13-IO.PA1@34
- net GND: now also JP20.58, JP20.60, X3.2; no longer C13.2, C14.2, C15.2, C16.2, C17.2, C18.2, C19.2, C20.2, C36.2, C37.2, C9.2, JP1.1, JP14.1, JP15.1, R22.1, SW1G$3.G, SW1G$4.G, U13-PWR.GND@114, U13-PWR.GND@17, U13-PWR.GND@48, U13-PWR.GND@55, U13-PWR.GND@58, U13-PWR.GND@80, U13-PWR.GNDA@10, U14.GND1, X4.2
- net HOST_GND: no longer C6.2, C7.2, U14.GND2, U17.GND, U17.GND_2
- net LDO1: now also JP20.5, JP20.59, JP20.6
- net LDO1_ENABLE: no longer U13-IO.PH3@32
- net LDO2: now also JP20.3, JP20.4
- net LDO2_ENABLE: no longer U13-IO.PH2@31
- net LDO3: now also JP20.1, JP20.2
- net LDO3_ENABLE: no longer U13-IO.PH1@30
- net LIN_CS: no longer U13-IO.PC5@24
- net LIN_RX: no longer U13-IO.PA6@40
- net LIN_TX: no longer U13-IO.PA7@41
- net M0S0: no longer U13-IO.PN0@107
- net M0S1: no longer U13-IO.PN1@108
- net M0S2: no longer U13-IO.PN2@109
- net M0S3: no longer U13-IO.PN3@110
- net M1S0: no longer U13-IO.PJ0@116
- net M1S1: no longer U13-IO.PJ1@117
- net M1S2: no longer U13-IO.PP1@119
- net M1S3: no longer U13-IO.PP0@118
- net M2S0: no longer U13-IO.PP2@103
- net M2S1: no longer U13-IO.PP3@104
- net M2S2: no longer U13-IO.PP4@105
- net M2S3: no longer U13-IO.PP5@106
- net N$10: now also JP20.11
- net N$100: now also JP20.38
- net N$101: now also JP20.40
- net N$102: now also JP20.42
- net N$103: now also JP20.44
- net N$104: now also JP20.46
- net N$105: now also JP20.48
- net N$106: now also JP20.50
- net N$107: now also JP20.52
- net N$108: now also JP20.54
- net N$109: now also JP20.56
- net N$11: now also JP20.13
- net N$12: now also JP20.15
- net N$13: now also JP20.17
- net N$14: now also JP20.19
- net N$15: now also JP20.21
- net N$16: now also JP20.23
- net N$17: now also JP20.25
- net N$18: now also JP20.27
- net N$19: now also JP20.29
- net N$20: now also JP20.31
- net N$21: now also JP20.33
- net N$22: now also JP20.35
- net N$24: now also JP20.37
- net N$26: now also JP20.39
- net N$27: now also JP20.41
- net N$28: now also JP20.43
- net N$29: now also JP20.45
- net N$30: now also JP20.47
- net N$31: now also JP20.49
- net N$32: now also JP20.51
- net N$37: now also JP20.53
- net N$38: now also JP20.55
- net N$39: now also JP20.57
- net N$4: now also SV2.2
- net N$43: now also SV1.14, SV2.14; no longer R18.1, SW1G$2.2
- net N$58: now also SV2.12
- net N$59: now also SV2.10
- net N$6: now also SV2.1
- net N$60: now also SV2.8
- net N$61: now also SV2.6
- net N$62: now also SV2.4
- net N$7: now also F1.1; no longer F1.2
- net N$75: now also SV2.13
- net N$76: now also SV2.11
- net N$77: now also SV2.9
- net N$78: now also SV2.7
- net N$79: now also SV2.5
- net N$8: now also JP20.7
- net N$80: now also SV2.3
- net N$85: now also JP20.8
- net N$86: now also JP20.10
- net N$87: now also JP20.12
- net N$88: now also JP20.14
- net N$89: now also JP20.16
- net N$9: now also JP20.9
- net N$90: now also JP20.18
- net N$91: now also JP20.20
- net N$92: now also JP20.22
- net N$93: now also JP20.24
- net N$94: now also JP20.26
- net N$95: now also JP20.28
- net N$96: now also JP20.30
- net N$97: now also JP20.32
- net N$98: now also JP20.34
- net N$99: now also JP20.36
- net NRESET: now also SV2.20
- net SWDCLK/TCLK/SCK: now also SV2.16
- net SWDIO/TMS: now also SV2.18
- net SWO/TDO/MOSI: now also SV2.15
- net TARGET_TCK/SWCLK: no longer U13-IO.PC0/TCK/SWCLK@100
- net TARGET_TDI: no longer U13-IO.PC2/TDI@98
- net TARGET_TDO/SWO: no longer U13-IO.PC3/TDO/SWO@97
- net TARGET_TMS/SWDIO: no longer U13-IO.PC1/TMS/SWDIO@99
- net TDI/MISO: now also SV2.17
- net TEST_FAIL: no longer U13-IO.PL5@86
- net TEST_PASS: no longer U13-IO.PL7@93
- net TEST_RUN: no longer U13-IO.PL6@94
- net TSTR_3V3: no longer C16.1, C17.1, C18.1, C19.1, R18.2, R19.2, R20.2, R21.2, R25.1, U13-PWR.VDD@101, U13-PWR.VDD@113, U13-PWR.VDD@122, U13-PWR.VDD@16, U13-PWR.VDD@26, U13-PWR.VDD@28, U13-PWR.VDD@39, U13-PWR.VDD@47, U13-PWR.VDD@51, U13-PWR.VDD@52, U13-PWR.VDD@69, U13-PWR.VDD@7, U13-PWR.VDD@79, U13-PWR.VDD@90, U13-PWR.VDDA@8, U13-PWR.VREFA+@9, U14.VDD1
- net TSTR_RX: no longer JP14.3, JP15.3, U13-IO.PC7@22, U14.VOA
- net TSTR_SCL: no longer U13-IO.PK4@63
- net TSTR_SDA: no longer U13-IO.PK5@62
- net TSTR_TX: no longer JP14.2, JP15.2, U13-IO.PC6@23, U14.VIB
- net USBD_N: no longer U17.USBDM
- net USBD_P: no longer U17.USBDP
- net VIN: now also F1.2; no longer F1.1
